File: schemat_i_inne/schemat/Niebieski/schemat_dip40.sch (KiCad schematic (older format))
At the start: 17 parts, among them J1 Conn_01x06_Female, SW1 Left, SW2 Up, SW3 Down, SW4 Right, SW5 Jump, SW6 Punch, SW7 SW_DIP_x01, U1 ATmega32A-AU, U2 WG12864B-STBL, U3 SD_card_reader, U4 L7805

Commit message: Schemat, scalenie i porzadki
->Zaktualizowano schemat
->Dodano skrypt manima.sh scalajacy poprzednie
->Dodano instrukcje tworzenia animacji
Parts:
- added Y1: 16Mhz, Crystal:Crystal_SMD_HC49-SD, symbol Device:Crystal
Connections:
- wire segments 163 -> 167
Changed lines of the file:
@@
 	5850 5600 6450 5600
 $Comp
-L power:GND #PWR?
+L power:GND #PWR09
 U 1 1 626E5836
 P 5550 4350
-F 0 "#PWR?" H 5550 4100 50  0001 C CNN
+F 0 "#PWR09" H 5550 4100 50  0001 C CNN
 F 1 "GND" V 5555 4222 50  0000 R CNN
 F 2 "" H 5550 4350 50  0001 C CNN
@@
 Wire Wire Line
 	5950 3200 5950 3650
+$Comp
+L Device:Crystal Y1
+U 1 1 626DC911
+P 1150 1900
+F 0 "Y1" V 1104 2031 50  0000 L CNN
+F 1 "16Mhz" V 1195 2031 50  0000 L CNN
+F 2 "Crystal:Crystal_SMD_HC49-SD" H 1150 1900 50  0001 C CNN
+F 3 "~" H 1150 1900 50  0001 C CNN
+	1    1150 1900
+	0    1    1    0
+$EndComp
+Wire Wire Line
+	1150 1750 1650 1750
+Wire Wire Line
+	1150 2050 1550 2050
+Wire Wire Line
+	1550 1950 1650 1950
+Wire Wire Line
+	1550 1950 1550 2050
 $EndSCHEMATC

Commit message: Zmieniono uklad symboli na plytce
Parts:
- added R2: 0R, Resistor_THT:R_Axial_DIN0309_L9.0mm_D3.2mm_P5.08mm_Vertical, symbol Device:R
Connections:
- wire segments 167 -> 161
Changed lines of the file:
@@
 	2250 1250 2250 900
 Wire Wire Line
-	8700 4600 3000 4600
-Wire Wire Line
 	8700 5150 7050 5150
 Wire Wire Line
@@
 	3650 4950 3650 4650
 Wire Wire Line
-	3650 4650 2850 4650
-Wire Wire Line
 	10700 4800 9900 4800
 Wire Wire Line
@@
 	3550 5050 3550 4750
 Wire Wire Line
-	3550 4750 2850 4750
-Wire Wire Line
-	6450 5600 9100 5600
-Wire Wire Line
-	9100 5600 9100 5350
-Connection ~ 6450 5600
-Wire Wire Line
-	9100 5600 9700 5600
-Wire Wire Line
-	9700 5600 9700 4850
-Connection ~ 9100 5600
-Wire Wire Line
-	9700 5600 10700 5600
-Wire Wire Line
-	10700 5600 10700 5150
-Connection ~ 9700 5600
-Wire Wire Line
-	10700 5600 11100 5600
-Wire Wire Line
-	11100 5600 11100 4800
-Connection ~ 10700 5600
-Wire Wire Line
-	9100 5150 9100 4600
-Connection ~ 9100 5150
-Wire Wire Line
-	9100 5350 8500 5350
-Wire Wire Line
 	8500 5350 8500 4850
-Connection ~ 9100 5350
-Wire Wire Line
-	9100 5350 9100 5150
 $Comp
 L schemat_dip40-rescue:WG12864B-STBL-schemat_dip40-rescue U2
@@
 	10150 1950 10150 5500
 Wire Wire Line
-	3000 4600 3000 4550
-Wire Wire Line
-	3000 4550 2850 4550
-Wire Wire Line
 	8650 4750 3800 4750
 Wire Wire Line
@@
 Wire Wire Line
 	3750 4550 3550 4550
-Wire Wire Line
-	3550 4550 3550 4450
-Wire Wire Line
-	3550 4450 2850 4450
 Wire Wire Line
 	2850 4350 3900 4350
@@
 Wire Wire Line
 	1550 1950 1550 2050
+Wire Wire Line
+	3550 4550 3550 4450
+Wire Wire Line
+	3550 4450 2850 4450
+Wire Wire Line
+	3650 4650 2850 4650
+Wire Wire Line
+	3550 4750 2850 4750
+Wire Wire Line
+	8700 4600 3000 4600
+Wire Wire Line
+	3000 4600 3000 4550
+Wire Wire Line
+	3000 4550 2850 4550
+$Comp
+L Device:R R2
+U 1 1 627CBEAE
+P 8150 5600
+F 0 "R2" V 7943 5600 50  0000 C CNN
+F 1 "0R" V 8034 5600 50  0000 C CNN
+F 2 "Resistor_THT:R_Axial_DIN0309_L9.0mm_D3.2mm_P5.08mm_Vertical" V 8080 5600 50  0001 C CNN
+F 3 "~" H 8150 5600 50  0001 C CNN
+	1    8150 5600
+	0    1    1    0
+$EndComp
+Wire Wire Line
+	8300 5600 9100 5600
+Wire Wire Line
+	8000 5600 6450 5600
+Connection ~ 6450 5600
+Wire Wire Line
+	9100 5150 9100 5600
+$Comp
+L power:GND #PWR0101
+U 1 1 627E1A64
+P 8500 5350
+F 0 "#PWR0101" H 8500 5100 50  0001 C CNN
+F 1 "GND" V 8505 5222 50  0000 R CNN
+F 2 "" H 8500 5350 50  0001 C CNN
+F 3 "" H 8500 5350 50  0001 C CNN
+	1    8500 5350
+	0    -1   -1   0
+$EndComp
+$Comp
+L power:GND #PWR0102
+U 1 1 627E22B0
+P 9100 4600
+F 0 "#PWR0102" H 9100 4350 50  0001 C CNN
+F 1 "GND" H 9105 4427 50  0000 C CNN
+F 2 "" H 9100 4600 50  0001 C CNN
+F 3 "" H 9100 4600 50  0001 C CNN
+	1    9100 4600
+	1    0    0    -1
+$EndComp
+$Comp
+L power:GND #PWR0104
+U 1 1 627E2F19
+P 11100 4800
+F 0 "#PWR0104" H 11100 4550 50  0001 C CNN
+F 1 "GND" H 11105 4627 50  0000 C CNN
+F 2 "" H 11100 4800 50  0001 C CNN
+F 3 "" H 11100 4800 50  0001 C CNN
+	1    11100 4800
+	1    0    0    -1
+$EndComp
+$Comp
+L power:GND #PWR0105
+U 1 1 627E3595
+P 10700 5150
+F 0 "#PWR0105" H 10700 4900 50  0001 C CNN
+F 1 "GND" H 10705 4977 50  0000 C CNN
+F 2 "" H 10700 5150 50  0001 C CNN
+F 3 "" H 10700 5150 50  0001 C CNN
+	1    10700 5150
+	1    0    0    -1
+$EndComp
+Wire Wire Line
+	9700 4850 9700 5600
+Wire Wire Line
+	9700 5600 9100 5600
+Connection ~ 9100 5600
 $EndSCHEMATC

Commit message: Dodane polaczenia
Dodano wszystkie polaczenia
Parts:
- removed R1, R2: 0R, Resistor_THT:R_Axial_DIN0309_L9.0mm_D3.2mm_P5.08mm_Vertical, symbol Device:R
- renumbered SW7 to SW1, SW1 to SW2, SW2 to SW3, SW3 to SW4, SW4 to SW5, SW5 to SW6, SW6 to SW7, U4 to U2, U2 to U3, U3 to U4
Connections:
- wire segments 161 -> 160
Changed lines of the file:
@@
 $EndDescr
 $Comp
-L schemat_dip40-rescue:SD_card_reader-Connector U3
+L schemat_dip40-rescue:SD_card_reader-Connector U4
 U 1 1 61D7A0EB
 P 7250 4000
-F 0 "U3" H 8028 4046 50  0000 L CNN
+F 0 "U4" H 8028 4046 50  0000 L CNN
 F 1 "SD_card_reader" H 8028 3955 50  0000 L CNN
 F 2 "Connector_Card:SD_Kyocera_145638009511859+" H 7200 4000 50  0001 C CNN
@@
 	3600 1300 3600 3550
 $Comp
-L power:VCC #PWR04
+L power:VCC #PWR08
 U 1 1 61D95FE0
 P 7850 1050
-F 0 "#PWR04" H 7850 900 50  0001 C CNN
+F 0 "#PWR08" H 7850 900 50  0001 C CNN
 F 1 "VCC" H 7865 1223 50  0000 C CNN
 F 2 "" H 7850 1050 50  0001 C CNN
@@
 $EndComp
 $Comp
-L power:GND #PWR05
+L power:GND #PWR010
 U 1 1 61D975F7
 P 8700 3200
-F 0 "#PWR05" H 8700 2950 50  0001 C CNN
+F 0 "#PWR010" H 8700 2950 50  0001 C CNN
 F 1 "GND" H 8705 3027 50  0000 C CNN
 F 2 "" H 8700 3200 50  0001 C CNN
@@
 Connection ~ 7850 1050
 $Comp
-L power:VCC #PWR01
+L power:VCC #PWR02
 U 1 1 61DB3E6A
 P 2250 900
-F 0 "#PWR01" H 2250 750 50  0001 C CNN
+F 0 "#PWR02" H 2250 750 50  0001 C CNN
 F 1 "VCC" H 2265 1073 50  0000 C CNN
 F 2 "" H 2250 900 50  0001 C CNN
@@
 Connection ~ 2250 900
 $Comp
-L power:GND #PWR03
+L power:GND #PWR05
 U 1 1 61DBB00B
 P 5850 6000
-F 0 "#PWR03" H 5850 5750 50  0001 C CNN
+F 0 "#PWR05" H 5850 5750 50  0001 C CNN
 F 1 "GND" H 5855 5827 50  0000 C CNN
 F 2 "" H 5850 6000 50  0001 C CNN
@@
 $EndComp
 $Comp
-L power:VCC #PWR02
+L power:VCC #PWR03
 U 1 1 61DBD527
 P 5450 3750
-F 0 "#PWR02" H 5450 3600 50  0001 C CNN
+F 0 "#PWR03" H 5450 3600 50  0001 C CNN
 F 1 "VCC" H 5465 3923 50  0000 C CNN
 F 2 "" H 5450 3750 50  0001 C CNN
@@
 	5450 3850 5450 3750
 Wire Wire Line
-	6300 4350 5850 4350
-Wire Wire Line
 	6450 5100 4000 5100
 Wire Wire Line
@@
 Wire Wire Line
 	3200 4250 3200 3050
-Wire Wire Line
-	6450 5500 10150 5500
-$Comp
-L Switch:SW_Push SW2
+$Comp
+L Switch:SW_Push SW3
 U 1 1 6261EEBB
 P 8900 4600
-F 0 "SW2" H 8900 4885 50  0000 C CNN
+F 0 "SW3" H 8900 4885 50  0000 C CNN
 F 1 "Up" H 8900 4794 50  0000 C CNN
 F 2 "Button_Switch_THT:SW_PUSH-12mm" H 8900 4800 50  0001 C CNN
@@
 $EndComp
 $Comp
-L Switch:SW_Push SW3
+L Switch:SW_Push SW4
 U 1 1 6261FEC3
 P 8900 5150
-F 0 "SW3" H 8900 5435 50  0000 C CNN
+F 0 "SW4" H 8900 5435 50  0000 C CNN
 F 1 "Down" H 8900 5344 50  0000 C CNN
 F 2 "Button_Switch_THT:SW_PUSH-12mm" H 8900 5350 50  0001 C CNN
@@
 $EndComp
 $Comp
-L Switch:SW_Push SW4
+L Switch:SW_Push SW5
 U 1 1 6262059D
 P 9500 4850
-F 0 "SW4" H 9500 5135 50  0000 C CNN
+F 0 "SW5" H 9500 5135 50  0000 C CNN
 F 1 "Right" H 9500 5044 50  0000 C CNN
 F 2 "Button_Switch_THT:SW_PUSH-12mm" H 9500 5050 50  0001 C CNN
@@
 $EndComp
 $Comp
-L Switch:SW_Push SW1
+L Switch:SW_Push SW2
 U 1 1 62620D64
 P 8300 4850
-F 0 "SW1" H 8300 5135 50  0000 C CNN
+F 0 "SW2" H 8300 5135 50  0000 C CNN
 F 1 "Left" H 8300 5044 50  0000 C CNN
 F 2 "Button_Switch_THT:SW_PUSH-12mm" H 8300 5050 50  0001 C CNN
@@
 $EndComp
 $Comp
-L Switch:SW_Push SW5
+L Switch:SW_Push SW6
 U 1 1 626213AA
 P 10500 5150
-F 0 "SW5" H 10500 5435 50  0000 C CNN
+F 0 "SW6" H 10500 5435 50  0000 C CNN
 F 1 "Jump" H 10500 5344 50  0000 C CNN
 F 2 "Button_Switch_THT:SW_PUSH-12mm" H 10500 5350 50  0001 C CNN
@@
 $EndComp
 $Comp
-L Switch:SW_Push SW6
+L Switch:SW_Push SW7
 U 1 1 6262299A
 P 10900 4800
-F 0 "SW6" H 10900 5085 50  0000 C CNN
+F 0 "SW7" H 10900 5085 50  0000 C CNN
 F 1 "Punch" H 10900 4994 50  0000 C CNN
 F 2 "Button_Switch_THT:SW_PUSH-12mm" H 10900 5000 50  0001 C CNN
@@
 	8500 5350 8500 4850
 $Comp
-L schemat_dip40-rescue:WG12864B-STBL-schemat_dip40-rescue U2
+L schemat_dip40-rescue:WG12864B-STBL-schemat_dip40-rescue U3
 U 1 1 6264714C
 P 6600 2300
-F 0 "U2" H 6600 3331 50  0000 C CNN
+F 0 "U3" H 6600 3331 50  0000 C CNN
 F 1 "WG12864B-STBL" H 6600 3240 50  0000 C CNN
 F 2 "Blue:WG12864BL" H 6600 2300 50  0001 C CNN
@@
 $EndComp
 $Comp
-L Regulator_Linear:L7805 U4
+L Regulator_Linear:L7805 U2
 U 1 1 62650285
 P 6100 6600
-F 0 "U4" H 6100 6842 50  0000 C CNN
+F 0 "U2" H 6100 6842 50  0000 C CNN
 F 1 "L7805" H 6100 6751 50  0000 C CNN
 F 2 "Package_TO_SOT_SMD:TO-263-2" H 6125 6450 50  0001 L CIN
@@
 $EndComp
 $Comp
-L Switch:SW_DIP_x01 SW7
+L Switch:SW_DIP_x01 SW1
 U 1 1 626527EA
 P 3250 6750
-F 0 "SW7" H 3250 7017 50  0000 C CNN
+F 0 "SW1" H 3250 7017 50  0000 C CNN
 F 1 "SW_DIP_x01" H 3250 6926 50  0000 C CNN
 F 2 "Connector_PinHeader_2.54mm:PinHeader_1x03_P2.54mm_Vertical" H 3250 6750 50  0001 C CNN
@@
 	2950 6600 2950 6750
 $Comp
-L power:VCC #PWR08
+L power:VCC #PWR07
 U 1 1 6266E18D
 P 6750 6650
-F 0 "#PWR08" H 6750 6500 50  0001 C CNN
+F 0 "#PWR07" H 6750 6500 50  0001 C CNN
 F 1 "VCC" H 6767 6823 50  0000 C CNN
 F 2 "" H 6750 6650 50  0001 C CNN
@@
 	6550 6650 6750 6650
 $Comp
-L power:GND #PWR07
+L power:GND #PWR06
 U 1 1 62676E00
 P 6000 6950
-F 0 "#PWR07" H 6000 6700 50  0001 C CNN
+F 0 "#PWR06" H 6000 6700 50  0001 C CNN
 F 1 "GND" H 6005 6777 50  0000 C CNN
 F 2 "" H 6000 6950 50  0001 C CNN
@@
 	6100 6950 6100 6900
 $Comp
-L power:GND #PWR06
+L power:GND #PWR01
 U 1 1 6268019B
 P 1150 7550
-F 0 "#PWR06" H 1150 7300 50  0001 C CNN
+F 0 "#PWR01" H 1150 7300 50  0001 C CNN
 F 1 "GND" H 1155 7377 50  0000 C CNN
 F 2 "" H 1150 7550 50  0001 C CNN
@@
 Wire Wire Line
 	2850 4350 3900 4350
-$Comp
-L Device:R R1
-U 1 1 626CB655
-P 5700 4350
-F 0 "R1" V 5493 4350 50  0000 C CNN
-F 1 "0R" V 5584 4350 50  0000 C CNN
-F 2 "Resistor_THT:R_Axial_DIN0309_L9.0mm_D3.2mm_P5.08mm_Vertical" V 5630 4350 50  0001 C CNN
-F 3 "~" H 5700 4350 50  0001 C CNN
-	1    5700 4350
-	0    1    1    0
-$EndComp
 Wire Wire Line
 	2250 5600 5850 5600
@@
 	5850 5600 6450 5600
 $Comp
-L power:GND #PWR09
+L power:GND #PWR04
 U 1 1 626E5836
 P 5550 4350
-F 0 "#PWR09" H 5550 4100 50  0001 C CNN
+F 0 "#PWR04" H 5550 4100 50  0001 C CNN
 F 1 "GND" V 5555 4222 50  0000 R CNN
 F 2 "" H 5550 4350 50  0001 C CNN
@@
 Wire Wire Line
 	3000 4550 2850 4550
-$Comp
-L Device:R R2
-U 1 1 627CBEAE
-P 8150 5600
-F 0 "R2" V 7943 5600 50  0000 C CNN
-F 1 "0R" V 8034 5600 50  0000 C CNN
-F 2 "Resistor_THT:R_Axial_DIN0309_L9.0mm_D3.2mm_P5.08mm_Vertical" V 8080 5600 50  0001 C CNN
-F 3 "~" H 8150 5600 50  0001 C CNN
-	1    8150 5600
-	0    1    1    0
-$EndComp
-Wire Wire Line
-	8300 5600 9100 5600
-Wire Wire Line
-	8000 5600 6450 5600
-Connection ~ 6450 5600
 Wire Wire Line
 	9100 5150 9100 5600
 $Comp
-L power:GND #PWR0101
+L power:GND #PWR09
 U 1 1 627E1A64
 P 8500 5350
-F 0 "#PWR0101" H 8500 5100 50  0001 C CNN
+F 0 "#PWR09" H 8500 5100 50  0001 C CNN
 F 1 "GND" V 8505 5222 50  0000 R CNN
 F 2 "" H 8500 5350 50  0001 C CNN
@@
 $EndComp
 $Comp
-L power:GND #PWR0102
+L power:GND #PWR011
 U 1 1 627E22B0
 P 9100 4600
-F 0 "#PWR0102" H 9100 4350 50  0001 C CNN
+F 0 "#PWR011" H 9100 4350 50  0001 C CNN
 F 1 "GND" H 9105 4427 50  0000 C CNN
 F 2 "" H 9100 4600 50  0001 C CNN
@@
 $EndComp
 $Comp
-L power:GND #PWR0104
+L power:GND #PWR013
 U 1 1 627E2F19
 P 11100 4800
-F 0 "#PWR0104" H 11100 4550 50  0001 C CNN
+F 0 "#PWR013" H 11100 4550 50  0001 C CNN
 F 1 "GND" H 11105 4627 50  0000 C CNN
 F 2 "" H 11100 4800 50  0001 C CNN
@@
 $EndComp
 $Comp
-L power:GND #PWR0105
+L power:GND #PWR012
 U 1 1 627E3595
 P 10700 5150
-F 0 "#PWR0105" H 10700 4900 50  0001 C CNN
+F 0 "#PWR012" H 10700 4900 50  0001 C CNN
 F 1 "GND" H 10705 4977 50  0000 C CNN
 F 2 "" H 10700 5150 50  0001 C CNN
@@
 Wire Wire Line
 	9700 5600 9100 5600
+Wire Wire Line
+	5550 4350 6300 4350
 Connection ~ 9100 5600
+Connection ~ 6450 5600
+Wire Wire Line
+	6450 5500 10150 5500
+Wire Wire Line
+	6450 5600 9100 5600
 $EndSCHEMATC

Commit message: Buzzer
Dodano buzzer
Parts:
- added BZ1: Buzzer, Buzzer_Beeper:Buzzer_12x9.5RM7.6, symbol Device:Buzzer
Connections:
- wire segments 160 -> 164
Changed lines of the file:
@@
 	3500 3350 2850 3350
 Wire Wire Line
-	2250 5250 2250 5600
+	2250 5250 2250 5300
 Wire Wire Line
 	2250 1250 2250 900
@@
 Wire Wire Line
 	6450 5600 9100 5600
+$Comp
+L Device:Buzzer BZ1
+U 1 1 627A142A
+P 2950 5400
+F 0 "BZ1" V 2908 5552 50  0000 L CNN
+F 1 "Buzzer" V 2999 5552 50  0000 L CNN
+F 2 "Buzzer_Beeper:Buzzer_12x9.5RM7.6" V 2925 5500 50  0001 C CNN
+F 3 "~" V 2925 5500 50  0001 C CNN
+	1    2950 5400
+	0    1    1    0
+$EndComp
+Wire Wire Line
+	2850 4950 3050 4950
+Wire Wire Line
+	3050 4950 3050 5300
+Wire Wire Line
+	2850 5300 2250 5300
+Connection ~ 2250 5300
+Wire Wire Line
+	2250 5300 2250 5600
 $EndSCHEMATC

Commit message: Kolejne zmiany w szchemacie i plytce
->Dodano gniazdo ethernetowe i adapter zamiast zlacza 6pin
 aby byla mozliwa komunikacja miedzy konsolami
->zmieniono rozmieszczenie przyciskow
->drobne poprawki sciezek
Parts:
- removed J1: Conn_01x06_Female, Connector_PinHeader_2.54mm:PinHeader_1x06_P2.54mm_Vertical, symbol Connector:Conn_01x06_Female
- added J1: Hole1, Connector_PinHeader_2.54mm:PinHeader_1x01_P2.54mm_Vertical, symbol Connector:Conn_01x01_Female
- added J2: Hole2, Connector_PinHeader_2.54mm:PinHeader_1x01_P2.54mm_Vertical, symbol Connector:Conn_01x01_Female
- added J3: Hole3, Connector_PinHeader_2.54mm:PinHeader_1x01_P2.54mm_Vertical, symbol Connector:Conn_01x01_Female
- added J4: Hole4, Connector_PinHeader_2.54mm:PinHeader_1x01_P2.54mm_Vertical, symbol Connector:Conn_01x01_Female
- added J5: RJ45, Connector_RJ:RJ45_Amphenol_54602-x08_Horizontal, symbol Connector:RJ45
- added R1: 0R, Resistor_THT:R_Axial_DIN0204_L3.6mm_D1.6mm_P2.54mm_Vertical, symbol Device:R
- U2: footprint Package_TO_SOT_SMD:TO-263-2 -> Package_TO_SOT_THT:TO-220-3_Vertical
Connections:
- wire segments 164 -> 189
Other:
- note removed: "GND\n"
- note removed: "MISO"
- note removed: "MOSI"
- note removed: "RST"
- note removed: "SCK\n"
- note removed: "USBASP programator"
- note removed: "VCC"
Changed lines of the file:
@@
 	1    0    0    -1
 $EndComp
-$Comp
-L Connector:Conn_01x06_Female J1
-U 1 1 61D899A2
-P 6650 5300
-F 0 "J1" H 6678 5276 50  0000 L CNN
-F 1 "Conn_01x06_Female" H 6678 5185 50  0000 L CNN
-F 2 "Connector_PinHeader_2.54mm:PinHeader_1x06_P2.54mm_Vertical" H 6650 5300 50  0001 C CNN
-F 3 "~" H 6650 5300 50  0001 C CNN
-	1    6650 5300
-	1    0    0    -1
-$EndComp
-Text Notes 6700 5850 0    50   ~ 0
-USBASP programator
-Text Notes 6800 5650 0    50   ~ 0
-GND\n
-Text Notes 6800 5550 0    50   ~ 0
-VCC
-Text Notes 6800 5450 0    50   ~ 0
-MOSI
-Text Notes 6800 5350 0    50   ~ 0
-MISO
-Text Notes 6800 5250 0    50   ~ 0
-SCK\n
-Text Notes 6800 5150 0    50   ~ 0
-RST
 Wire Wire Line
 	6100 2150 5550 2150
@@
 	5450 3850 5450 3750
 Wire Wire Line
-	6450 5100 4000 5100
-Wire Wire Line
 	4000 5100 4000 5800
 Wire Wire Line
@@
 Wire Wire Line
 	1350 5800 1350 1550
-Wire Wire Line
-	6450 5200 3300 5200
-Wire Wire Line
-	3300 5200 3300 4150
-Wire Wire Line
-	6450 5300 3200 5300
-Wire Wire Line
-	3200 5300 3200 4250
-Wire Wire Line
-	6450 5400 3100 5400
 Wire Wire Line
 	3100 5400 3100 4050
@@
 Wire Wire Line
 	6300 4250 3200 4250
-Connection ~ 3200 4250
 Wire Wire Line
 	3200 4250 3200 3050
@@
 	3750 4850 3750 4550
 Wire Wire Line
-	10300 5150 9400 5150
-Wire Wire Line
 	9400 5150 9400 4950
 Wire Wire Line
@@
 Wire Wire Line
 	3650 4950 3650 4650
-Wire Wire Line
-	10700 4800 9900 4800
-Wire Wire Line
-	9900 4800 9900 5050
-Wire Wire Line
-	9900 5050 3550 5050
 Wire Wire Line
 	3550 5050 3550 4750
@@
 F 0 "U2" H 6100 6842 50  0000 C CNN
 F 1 "L7805" H 6100 6751 50  0000 C CNN
-F 2 "Package_TO_SOT_SMD:TO-263-2" H 6125 6450 50  0001 L CIN
+F 2 "Package_TO_SOT_THT:TO-220-3_Vertical" H 6125 6450 50  0001 L CIN
 F 3 "http://www.st.com/content/ccc/resource/technical/document/datasheet/41/4f/b3/b0/12/d4/47/88/CD00000444.pdf/files/CD00000444.pdf/jcr:content/translations/en.CD00000444.pdf" H 6100 6550 50  0001 C CNN
 	1    6100 6600
@@
 Connection ~ 10150 1950
 Wire Wire Line
-	10150 1950 10150 5500
-Wire Wire Line
 	8650 4750 3800 4750
 Wire Wire Line
@@
 Wire Wire Line
 	5850 6000 5850 5600
-Connection ~ 5850 5600
-Wire Wire Line
-	5850 5600 6450 5600
 $Comp
 L power:GND #PWR04
@@
 	3000 4550 2850 4550
 Wire Wire Line
-	9100 5150 9100 5600
+	9100 5150 9100 5500
 $Comp
 L power:GND #PWR09
@@
 Wire Wire Line
 	9700 4850 9700 5600
-Wire Wire Line
-	9700 5600 9100 5600
-Wire Wire Line
-	5550 4350 6300 4350
-Connection ~ 9100 5600
-Connection ~ 6450 5600
-Wire Wire Line
-	6450 5500 10150 5500
-Wire Wire Line
-	6450 5600 9100 5600
 $Comp
 L Device:Buzzer BZ1
@@
 Wire Wire Line
 	2250 5300 2250 5600
+Wire Wire Line
+	9100 5600 9700 5600
+Wire Wire Line
+	3200 4250 3200 5200
+Connection ~ 3200 4250
+Wire Wire Line
+	3300 4150 3300 5300
+Wire Wire Line
+	5850 5600 5850 5500
+Connection ~ 5850 5600
+Connection ~ 9100 5500
+Wire Wire Line
+	9100 5500 9100 5600
+$Comp
+L power:VCC #PWR0101
+U 1 1 628A7A02
+P 6300 5800
+F 0 "#PWR0101" H 6300 5650 50  0001 C CNN
+F 1 "VCC" H 6318 5973 50  0000 C CNN
+F 2 "" H 6300 5800 50  0001 C CNN
+F 3 "" H 6300 5800 50  0001 C CNN
+	1    6300 5800
+	-1   0    0    1
+$EndComp
+Wire Wire Line
+	6300 5800 6300 5600
+Wire Wire Line
+	3650 5300 3650 5200
+Wire Wire Line
+	3650 5200 3200 5200
+Wire Wire Line
+	3850 5200 3850 5250
+Wire Wire Line
+	3850 5250 3550 5250
+Wire Wire Line
+	3550 5250 3550 5300
+Wire Wire Line
+	3550 5300 3300 5300
+$Comp
+L Connector:Conn_01x01_Female J1
+U 1 1 627D6C2D
+P 10650 800
+F 0 "J1" H 10678 826 50  0000 L CNN
+F 1 "Hole1" H 10678 735 50  0000 L CNN
+F 2 "Connector_PinHeader_2.54mm:PinHeader_1x01_P2.54mm_Vertical" H 10650 800 50  0001 C CNN
+F 3 "~" H 10650 800 50  0001 C CNN
+	1    10650 800
+	1    0    0    -1
+$EndComp
+$Comp
+L Connector:Conn_01x01_Female J2
+U 1 1 627D7CE4
+P 10650 950
+F 0 "J2" H 10678 976 50  0000 L CNN
+F 1 "Hole2" H 10678 885 50  0000 L CNN
+F 2 "Connector_PinHeader_2.54mm:PinHeader_1x01_P2.54mm_Vertical" H 10650 950 50  0001 C CNN
+F 3 "~" H 10650 950 50  0001 C CNN
+	1    10650 950
+	1    0    0    -1
+$EndComp
+$Comp
+L Connector:Conn_01x01_Female J3
+U 1 1 627D8D77
+P 10650 1150
+F 0 "J3" H 10678 1176 50  0000 L CNN
+F 1 "Hole3" H 10678 1085 50  0000 L CNN
+F 2 "Connector_PinHeader_2.54mm:PinHeader_1x01_P2.54mm_Vertical" H 10650 1150 50  0001 C CNN
+F 3 "~" H 10650 1150 50  0001 C CNN
+	1    10650 1150
+	1    0    0    -1
+$EndComp
+$Comp
+L Connector:Conn_01x01_Female J4
+U 1 1 627D9436
+P 10650 1300
+F 0 "J4" H 10678 1326 50  0000 L CNN
+F 1 "Hole4" H 10678 1235 50  0000 L CNN
+F 2 "Connector_PinHeader_2.54mm:PinHeader_1x01_P2.54mm_Vertical" H 10650 1300 50  0001 C CNN
+F 3 "~" H 10650 1300 50  0001 C CNN
+	1    10650 1300
+	1    0    0    -1
+$EndComp
+Wire Wire Line
+	9250 5200 9250 3750
+Wire Wire Line
+	9800 5400 9800 3650
+Wire Wire Line
+	10300 5150 9400 5150
+Wire Wire Line
+	9750 5100 9750 3350
+Wire Wire Line
+	9750 3350 9650 3350
+Wire Wire Line
+	9650 3350 9650 2950
+Wire Wire Line
+	10150 5800 6500 5800
+Wire Wire Line
+	6500 5800 6500 5600
+Wire Wire Line
+	10150 1950 10150 5800
+$Comp
+L Connector:RJ45 J5
+U 1 1 6286835F
+P 9450 2550
+F 0 "J5" V 9461 3080 50  0000 L CNN
+F 1 "RJ45" V 9552 3080 50  0000 L CNN
+F 2 "Connector_RJ:RJ45_Amphenol_54602-x08_Horizontal" V 9450 2575 50  0001 C CNN
+F 3 "~" V 9450 2575 50  0001 C CNN
+	1    9450 2550
+	0    1    1    0
+$EndComp
+$Comp
+L power:VCC #PWR0103
+U 1 1 62891AEF
+P 9150 3100
+F 0 "#PWR0103" H 9150 2950 50  0001 C CNN
+F 1 "VCC" H 9168 3273 50  0000 C CNN
+F 2 "" H 9150 3100 50  0001 C CNN
+F 3 "" H 9150 3100 50  0001 C CNN
+	1    9150 3100
+	-1   0    0    1
+$EndComp
+Wire Wire Line
+	9150 2950 9150 3100
+Wire Wire Line
+	9250 3100 9250 2950
+Wire Wire Line
+	9550 3750 9550 2950
+Wire Wire Line
+	9250 3750 9550 3750
+Wire Wire Line
+	9900 3550 9450 3550
+Wire Wire Line
+	9450 3550 9450 2950
+Wire Wire Line
+	9800 3650 9350 3650
+Wire Wire Line
+	9350 3650 9350 2950
+$Comp
+L power:GND #PWR0102
+U 1 1 62A2A7B3
+P 9250 3100
+F 0 "#PWR0102" H 9250 2850 50  0001 C CNN
+F 1 "GND" H 9255 2927 50  0000 C CNN
+F 2 "" H 9250 3100 50  0001 C CNN
+F 3 "" H 9250 3100 50  0001 C CNN
+	1    9250 3100
+	1    0    0    -1
+$EndComp
+Wire Wire Line
+	10050 5050 10050 4800
+Wire Wire Line
+	10050 4800 10700 4800
+Wire Wire Line
+	3550 5050 10050 5050
+Wire Wire Line
+	9900 3550 9900 5300
+Wire Wire Line
+	4000 5100 9750 5100
+Wire Wire Line
+	3850 5200 9250 5200
+Wire Wire Line
+	3650 5300 9900 5300
+Wire Wire Line
+	3100 5400 9800 5400
+Wire Wire Line
+	5850 5500 9100 5500
+Wire Wire Line
+	6300 5600 6500 5600
+$Comp
+L Device:R R1
+U 1 1 62A64D65
+P 6000 4350
+F 0 "R1" V 5793 4350 50  0000 C CNN
+F 1 "0R" V 5884 4350 50  0000 C CNN
+F 2 "Resistor_THT:R_Axial_DIN0204_L3.6mm_D1.6mm_P2.54mm_Vertical" V 5930 4350 50  0001 C CNN
+F 3 "~" H 6000 4350 50  0001 C CNN
+	1    6000 4350
+	0    1    1    0
+$EndComp
+Wire Wire Line
+	5550 4350 5850 4350
+Wire Wire Line
+	6150 4350 6300 4350
 $EndSCHEMATC
