File: schemat_i_inne/schemat/Niebieski/schemat_dip40.sch (KiCad schematic (older format))
At the start: 23 parts, among them J1 Hole1, J2 Hole2, J3 Hole3, J4 Hole4, J5 RJ45, SW1 SW_DIP_x01, SW2 Left, SW3 Up, SW4 Down, SW5 Right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

Commit message: Awful, but should work XD
Strasznie brzydko, wszystkie sciezki do poprawy graficznej.
Zamieniono przyciski tak aby były w dobrych miejscach
Connections:
- net at SW3.1: now also U1.43 (PB3); no longer U1.32 (PA5)
- net at SW4.1: now also U1.41 (PB1); no longer U1.35 (PA2)
- net at SW5.1: now also U1.42 (PB2); no longer U1.34 (PA3)
- net at SW2.1: now also U1.44 (PB4); no longer U1.33 (PA4)
- net at SW6.1: now also U1.35 (PA2); no longer U1.43 (PB3)
- net at SW7.1: now also U1.34 (PA3); no longer U1.44 (PB4)
Changed lines of the file:
@@
 $EndComp
 Wire Wire Line
-	6700 4650 6700 1750
+	6700 4650 6700 2200
 Wire Wire Line
-	6200 4350 6200 1950
+	6200 4350 6200 2300
 Wire Wire Line
 	7400 4350 7400 1850
-Wire Wire Line
-	7400 1850 2850 1850
 Wire Wire Line
 	6800 4100 6800 2050
@@
 Wire Wire Line
 	3800 3900 3800 3850
-Wire Wire Line
-	6800 2050 2850 2050
-Wire Wire Line
-	6200 1950 2850 1950
-Wire Wire Line
-	6700 1750 2850 1750
 $Comp
 L schemat_dip40-rescue:SD_card_reader-Connector U4
@@
 	8700 4350 8700 2500
 Wire Wire Line
-	8700 2500 4600 2500
+	8300 2450 8300 4700
 Wire Wire Line
-	4600 2500 4600 2850
+	4250 2450 4250 1750
 Wire Wire Line
-	4600 2850 2850 2850
+	4250 1750 2850 1750
 Wire Wire Line
-	8300 2450 4550 2450
+	4250 2450 8300 2450
 Wire Wire Line
-	4550 2450 4550 2750
+	4150 2500 4150 1850
 Wire Wire Line
-	4550 2750 2850 2750
+	4150 1850 2850 1850
 Wire Wire Line
-	8300 2450 8300 4700
+	4150 2500 8700 2500
+Wire Wire Line
+	6200 2300 4500 2300
+Wire Wire Line
+	4500 2300 4500 2850
+Wire Wire Line
+	6700 2200 4450 2200
+Wire Wire Line
+	6800 2050 4350 2050
+Wire Wire Line
+	7400 1850 4300 1850
+Wire Wire Line
+	4300 1850 4300 2650
+Wire Wire Line
+	4450 2200 4450 2550
+Wire Wire Line
+	4450 2550 2850 2550
+Wire Wire Line
+	4500 2850 2850 2850
+Wire Wire Line
+	4300 2650 2850 2650
+Wire Wire Line
+	4350 2750 2850 2750
+Wire Wire Line
+	4350 2050 4350 2750
 $EndSCHEMATC
