File: schemat_i_inne/schemat/Niebieski/schemat.sch (KiCad schematic (older format))
At the start: 23 parts, among them J1 Hole1, J2 Hole2, J3 Hole3, J4 Hole4, J5 RJ45, SW1 SW_DIP_x01, SW2 Left, SW3 Up, SW4 Down, SW5 Right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

Commit message: New branch konwerter started
Parts:
- added J?: SD_Card, symbol Connector:SD_Card
Changed lines of the file:
@@
 Wire Wire Line
 	4350 2050 4350 2750
+$Comp
+L Connector:SD_Card J?
+U 1 1 629A5D92
+P 8200 1150
+F 0 "J?" H 8200 1815 50  0000 C CNN
+F 1 "SD_Card" H 8200 1724 50  0000 C CNN
+F 2 "" H 8200 1150 50  0001 C CNN
+F 3 "http://portal.fciconnect.com/Comergent//fci/drawing/10067847.pdf" H 8200 1150 50  0001 C CNN
+	1    8200 1150
+	1    0    0    -1
+$EndComp
 $EndSCHEMATC
