File: schemat_i_inne/schemat/konwerter/karta/karta.kicad_pcb (KiCad board)
At the start: 2 copper layers, 30 x 35.6 mm, 2 parts, among them J1 Conn_01x06_Male, U1 SD

Commit message: Dodano by KK i przygotowano do produkcji
Parts:
- added J1: Conn_01x06_Male, Connector_PinHeader_2.54mm:PinHeader_1x06_P2.54mm_Vertical, B.Cu at (230.6, 169.9)
- added J1: Conn_01x06_Male, Connector_PinHeader_2.54mm:PinHeader_1x06_P2.54mm_Vertical, B.Cu at (124.0, 115.3)
- added J1: Conn_01x06_Male, Connector_PinHeader_2.54mm:PinHeader_1x06_P2.54mm_Vertical, B.Cu at (89.7, 115.3)
- added J1: Conn_01x06_Male, Connector_PinHeader_2.54mm:PinHeader_1x06_P2.54mm_Vertical, B.Cu at (19.8, 114.0)
- added J1: Conn_01x06_Male, Connector_PinHeader_2.54mm:PinHeader_1x06_P2.54mm_Vertical, B.Cu at (195.1, 115.3)
- added J1: Conn_01x06_Male, Connector_PinHeader_2.54mm:PinHeader_1x06_P2.54mm_Vertical, B.Cu at (55.4, 114.0)
- added J1: Conn_01x06_Male, Connector_PinHeader_2.54mm:PinHeader_1x06_P2.54mm_Vertical, B.Cu at (230.6, 60.7)
- added J1: Conn_01x06_Male, Connector_PinHeader_2.54mm:PinHeader_1x06_P2.54mm_Vertical, B.Cu at (159.5, 60.7)
- added J1: Conn_01x06_Male, Connector_PinHeader_2.54mm:PinHeader_1x06_P2.54mm_Vertical, B.Cu at (195.1, 60.7)
- added J1: Conn_01x06_Male, Connector_PinHeader_2.54mm:PinHeader_1x06_P2.54mm_Vertical, B.Cu at (124.0, 60.7)
- added J1: Conn_01x06_Male, Connector_PinHeader_2.54mm:PinHeader_1x06_P2.54mm_Vertical, B.Cu at (89.7, 60.7)
- added J1: Conn_01x06_Male, Connector_PinHeader_2.54mm:PinHeader_1x06_P2.54mm_Vertical, B.Cu at (159.5, 169.9)
- added J1: Conn_01x06_Male, Connector_PinHeader_2.54mm:PinHeader_1x06_P2.54mm_Vertical, B.Cu at (55.4, 59.4)
- added J1: Conn_01x06_Male, Connector_PinHeader_2.54mm:PinHeader_1x06_P2.54mm_Vertical, B.Cu at (124.0, 169.9)
- added J1: Conn_01x06_Male, Connector_PinHeader_2.54mm:PinHeader_1x06_P2.54mm_Vertical, B.Cu at (89.7, 169.9)
- added J1: Conn_01x06_Male, Connector_PinHeader_2.54mm:PinHeader_1x06_P2.54mm_Vertical, B.Cu at (19.8, 168.7)
- added J1: Conn_01x06_Male, Connector_PinHeader_2.54mm:PinHeader_1x06_P2.54mm_Vertical, B.Cu at (195.1, 169.9)
- added J1: Conn_01x06_Male, Connector_PinHeader_2.54mm:PinHeader_1x06_P2.54mm_Vertical, B.Cu at (55.4, 168.7)
- added J1: Conn_01x06_Male, Connector_PinHeader_2.54mm:PinHeader_1x06_P2.54mm_Vertical, B.Cu at (230.6, 115.3)
- added J1: Conn_01x06_Male, Connector_PinHeader_2.54mm:PinHeader_1x06_P2.54mm_Vertical, B.Cu at (159.5, 115.3)
- added U1: SD, Connector_Card:SD_Kyocera_145638009511859+, F.Cu at (29.3, 156.2)
- added U1: SD, Connector_Card:SD_Kyocera_145638009511859+, F.Cu at (169.0, 102.9)
- added U1: SD, Connector_Card:SD_Kyocera_145638009511859+, F.Cu at (133.4, 102.9)
- added U1: SD, Connector_Card:SD_Kyocera_145638009511859+, F.Cu at (99.1, 102.9)
- added U1: SD, Connector_Card:SD_Kyocera_145638009511859+, F.Cu at (64.8, 101.6)
- added U1: SD, Connector_Card:SD_Kyocera_145638009511859+, F.Cu at (204.5, 102.9)
- added U1: SD, Connector_Card:SD_Kyocera_145638009511859+, F.Cu at (240.1, 48.3)
- added U1: SD, Connector_Card:SD_Kyocera_145638009511859+, F.Cu at (169.0, 48.3)
- added U1: SD, Connector_Card:SD_Kyocera_145638009511859+, F.Cu at (204.5, 48.3)
- added U1: SD, Connector_Card:SD_Kyocera_145638009511859+, F.Cu at (133.4, 48.3)
- added U1: SD, Connector_Card:SD_Kyocera_145638009511859+, F.Cu at (99.1, 48.3)
- added U1: SD, Connector_Card:SD_Kyocera_145638009511859+, F.Cu at (240.1, 157.5)
- added U1: SD, Connector_Card:SD_Kyocera_145638009511859+, F.Cu at (64.8, 47.0)
- added U1: SD, Connector_Card:SD_Kyocera_145638009511859+, F.Cu at (169.0, 157.5)
- added U1: SD, Connector_Card:SD_Kyocera_145638009511859+, F.Cu at (133.4, 157.5)
- added U1: SD, Connector_Card:SD_Kyocera_145638009511859+, F.Cu at (99.1, 157.5)
- added U1: SD, Connector_Card:SD_Kyocera_145638009511859+, F.Cu at (64.8, 156.2)
- added U1: SD, Connector_Card:SD_Kyocera_145638009511859+, F.Cu at (204.5, 157.5)
- added U1: SD, Connector_Card:SD_Kyocera_145638009511859+, F.Cu at (29.3, 101.6)
- added U1: SD, Connector_Card:SD_Kyocera_145638009511859+, F.Cu at (240.1, 102.9)
Routing:
- net (no net): track 0.00 -> 1896.4 mm
Other:
- board size 30 x 35.6 mm -> 240.8 x 146.1 mm
- board text added: "by KK"

Commit message: Kolejna zmiana konwertera
-> poprzedni konwerter dzialal, ale nie wzialem
pod uwage droputu na MOSFETach, wiec poziomy logiczne i tak
sie nie zgadzaly

-> zmieniony konwerter z gotowa plytka, dzialajacy juz na
normalnych zasadach
Other:
- net class Default removed
