File: schemat_i_inne/schemat/konwerter/karta+konwerter/konwerter.kicad_pcb (KiCad board)
At the start: 2 copper layers, 269.2 x 182.9 mm, 13 parts, among them J1 Conn_01x06_Male, U1 IRF7476, U2 LM1117-1.8, U3 IRF7476, U4 IRF7476, U5 IRF7476, U6 SD

Commit message: Kolejna zmiana konwertera
-> poprzedni konwerter dzialal, ale nie wzialem
pod uwage droputu na MOSFETach, wiec poziomy logiczne i tak
sie nie zgadzaly

-> zmieniony konwerter z gotowa plytka, dzialajacy juz na
normalnych zasadach
Other:
- net class Default removed
