File: schemat_i_inne/schemat/konwerter/konwerter/konwerter.kicad_pcb (KiCad board)
At the start: 2 copper layers, 269.2 x 182.9 mm, 8 parts, among them J1 Conn_01x03_Male, U1 IRF7476

Commit message: Gotowa plytka karty z konwerterem
Parts:
- removed the J1 at (63.5, 17.5)
- removed the J1 at (48.3, 17.5)
- removed the J1 at (33.0, 17.5)
- removed the J1 at (17.8, 17.5)
- removed the U1 at (69.9, 19.7)
- removed the U1 at (54.7, 19.7)
- removed the U1 at (39.5, 19.7)
- removed the U1 at (24.2, 19.7)
- added C1: 100N, Connector_PinHeader_2.54mm:PinHeader_1x02_P2.54mm_Vertical, B.Cu at (210.1, 157.9)
- added C1: 100N, Connector_PinHeader_2.54mm:PinHeader_1x02_P2.54mm_Vertical, B.Cu at (57.7, 84.2)
- added C1: 100N, Connector_PinHeader_2.54mm:PinHeader_1x02_P2.54mm_Vertical, B.Cu at (260.9, 157.9)
- added C1: 100N, Connector_PinHeader_2.54mm:PinHeader_1x02_P2.54mm_Vertical, B.Cu at (57.7, 157.9)
- added C1: 100N, Connector_PinHeader_2.54mm:PinHeader_1x02_P2.54mm_Vertical, B.Cu at (108.5, 157.9)
- added C1: 100N, Connector_PinHeader_2.54mm:PinHeader_1x02_P2.54mm_Vertical, B.Cu at (159.3, 157.9)
- added C1: 100N, Connector_PinHeader_2.54mm:PinHeader_1x02_P2.54mm_Vertical, B.Cu at (260.9, 84.2)
- added C1: 100N, Connector_PinHeader_2.54mm:PinHeader_1x02_P2.54mm_Vertical, B.Cu at (210.1, 84.2)
- added C1: 100N, Connector_PinHeader_2.54mm:PinHeader_1x02_P2.54mm_Vertical, B.Cu at (159.3, 84.2)
- added C1: 100N, Connector_PinHeader_2.54mm:PinHeader_1x02_P2.54mm_Vertical, B.Cu at (108.5, 84.2)
- added C2: 100N, Connector_PinHeader_2.54mm:PinHeader_1x02_P2.54mm_Vertical, B.Cu at (57.9, 148.3)
- added C2: 100N, Connector_PinHeader_2.54mm:PinHeader_1x02_P2.54mm_Vertical, B.Cu at (57.9, 74.6)
- added C2: 100N, Connector_PinHeader_2.54mm:PinHeader_1x02_P2.54mm_Vertical, B.Cu at (261.1, 148.3)
- added C2: 100N, Connector_PinHeader_2.54mm:PinHeader_1x02_P2.54mm_Vertical, B.Cu at (210.3, 148.3)
- added C2: 100N, Connector_PinHeader_2.54mm:PinHeader_1x02_P2.54mm_Vertical, B.Cu at (159.5, 148.3)
- added C2: 100N, Connector_PinHeader_2.54mm:PinHeader_1x02_P2.54mm_Vertical, B.Cu at (108.7, 148.3)
- added C2: 100N, Connector_PinHeader_2.54mm:PinHeader_1x02_P2.54mm_Vertical, B.Cu at (261.1, 74.6)
- added C2: 100N, Connector_PinHeader_2.54mm:PinHeader_1x02_P2.54mm_Vertical, B.Cu at (210.3, 74.6)
- added C2: 100N, Connector_PinHeader_2.54mm:PinHeader_1x02_P2.54mm_Vertical, B.Cu at (159.5, 74.6)
- added C2: 100N, Connector_PinHeader_2.54mm:PinHeader_1x02_P2.54mm_Vertical, B.Cu at (108.7, 74.6)
- added D1: 4,7V, Diode_THT:D_DO-41_SOD81_P7.62mm_Horizontal, F.Cu at (42.8, 143.0)
- added D1: 4,7V, Diode_THT:D_DO-41_SOD81_P7.62mm_Horizontal, F.Cu at (42.8, 69.4)
- added D1: 4,7V, Diode_THT:D_DO-41_SOD81_P7.62mm_Horizontal, F.Cu at (144.4, 143.0)
- added D1: 4,7V, Diode_THT:D_DO-41_SOD81_P7.62mm_Horizontal, F.Cu at (246.0, 143.0)
- added D1: 4,7V, Diode_THT:D_DO-41_SOD81_P7.62mm_Horizontal, F.Cu at (195.2, 143.0)
- added D1: 4,7V, Diode_THT:D_DO-41_SOD81_P7.62mm_Horizontal, F.Cu at (93.6, 143.0)
- added D1: 4,7V, Diode_THT:D_DO-41_SOD81_P7.62mm_Horizontal, F.Cu at (246.0, 69.4)
- added D1: 4,7V, Diode_THT:D_DO-41_SOD81_P7.62mm_Horizontal, F.Cu at (195.2, 69.4)
- added D1: 4,7V, Diode_THT:D_DO-41_SOD81_P7.62mm_Horizontal, F.Cu at (144.4, 69.4)
- added D1: 4,7V, Diode_THT:D_DO-41_SOD81_P7.62mm_Horizontal, F.Cu at (93.6, 69.4)
- added J1: Conn_01x06_Male, Connector_PinHeader_2.54mm:PinHeader_1x06_P2.54mm_Vertical, B.Cu at (73.1, 154.5)
- added J1: Conn_01x06_Male, Connector_PinHeader_2.54mm:PinHeader_1x06_P2.54mm_Vertical, B.Cu at (22.3, 80.9)
- added J1: Conn_01x06_Male, Connector_PinHeader_2.54mm:PinHeader_1x06_P2.54mm_Vertical, B.Cu at (123.9, 154.5)
- added J1: Conn_01x06_Male, Connector_PinHeader_2.54mm:PinHeader_1x06_P2.54mm_Vertical, B.Cu at (174.7, 154.5)
- added J1: Conn_01x06_Male, Connector_PinHeader_2.54mm:PinHeader_1x06_P2.54mm_Vertical, B.Cu at (225.5, 154.5)
- added J1: Conn_01x06_Male, Connector_PinHeader_2.54mm:PinHeader_1x06_P2.54mm_Vertical, B.Cu at (22.3, 154.5)
- added J1: Conn_01x06_Male, Connector_PinHeader_2.54mm:PinHeader_1x06_P2.54mm_Vertical, B.Cu at (225.5, 80.9)
- added J1: Conn_01x06_Male, Connector_PinHeader_2.54mm:PinHeader_1x06_P2.54mm_Vertical, B.Cu at (174.7, 80.9)
- added J1: Conn_01x06_Male, Connector_PinHeader_2.54mm:PinHeader_1x06_P2.54mm_Vertical, B.Cu at (123.9, 80.9)
- added J1: Conn_01x06_Male, Connector_PinHeader_2.54mm:PinHeader_1x06_P2.54mm_Vertical, B.Cu at (73.1, 80.9)
- added J3: Micro_SD_Card, Connector_Card:SD_Kyocera_145638009511859+, F.Cu at (188.5, 127.0)
- added J3: Micro_SD_Card, Connector_Card:SD_Kyocera_145638009511859+, F.Cu at (36.1, 53.3)
- added J3: Micro_SD_Card, Connector_Card:SD_Kyocera_145638009511859+, F.Cu at (239.3, 127.0)
- added J3: Micro_SD_Card, Connector_Card:SD_Kyocera_145638009511859+, F.Cu at (36.1, 127.0)
- added J3: Micro_SD_Card, Connector_Card:SD_Kyocera_145638009511859+, F.Cu at (137.7, 127.0)
- added J3: Micro_SD_Card, Connector_Card:SD_Kyocera_145638009511859+, F.Cu at (86.9, 127.0)
- added J3: Micro_SD_Card, Connector_Card:SD_Kyocera_145638009511859+, F.Cu at (239.3, 53.3)
- added J3: Micro_SD_Card, Connector_Card:SD_Kyocera_145638009511859+, F.Cu at (188.5, 53.3)
- added J3: Micro_SD_Card, Connector_Card:SD_Kyocera_145638009511859+, F.Cu at (137.7, 53.3)
- added J3: Micro_SD_Card, Connector_Card:SD_Kyocera_145638009511859+, F.Cu at (86.9, 53.3)
- added R1: 10K, Resistor_SMD:R_0805_2012Metric_Pad1.15x1.40mm_HandSolder, F.Cu at (139.1, 140.6)
- added R1: 10K, Resistor_SMD:R_0805_2012Metric_Pad1.15x1.40mm_HandSolder, F.Cu at (37.5, 66.9)
- added R1: 10K, Resistor_SMD:R_0805_2012Metric_Pad1.15x1.40mm_HandSolder, F.Cu at (189.9, 140.6)
- added R1: 10K, Resistor_SMD:R_0805_2012Metric_Pad1.15x1.40mm_HandSolder, F.Cu at (240.7, 140.6)
- added R1: 10K, Resistor_SMD:R_0805_2012Metric_Pad1.15x1.40mm_HandSolder, F.Cu at (88.3, 140.6)
- added R1: 10K, Resistor_SMD:R_0805_2012Metric_Pad1.15x1.40mm_HandSolder, F.Cu at (37.5, 140.6)
- added R1: 10K, Resistor_SMD:R_0805_2012Metric_Pad1.15x1.40mm_HandSolder, F.Cu at (240.7, 66.9)
- added R1: 10K, Resistor_SMD:R_0805_2012Metric_Pad1.15x1.40mm_HandSolder, F.Cu at (189.9, 66.9)
- added R1: 10K, Resistor_SMD:R_0805_2012Metric_Pad1.15x1.40mm_HandSolder, F.Cu at (139.1, 66.9)
- added R1: 10K, Resistor_SMD:R_0805_2012Metric_Pad1.15x1.40mm_HandSolder, F.Cu at (88.3, 66.9)
- added R2: 10K, Resistor_SMD:R_0805_2012Metric_Pad1.15x1.40mm_HandSolder, F.Cu at (92.5, 154.4)
- added R2: 10K, Resistor_SMD:R_0805_2012Metric_Pad1.15x1.40mm_HandSolder, F.Cu at (41.7, 80.7)
- added R2: 10K, Resistor_SMD:R_0805_2012Metric_Pad1.15x1.40mm_HandSolder, F.Cu at (244.9, 154.4)
- added R2: 10K, Resistor_SMD:R_0805_2012Metric_Pad1.15x1.40mm_HandSolder, F.Cu at (143.3, 154.4)
- added R2: 10K, Resistor_SMD:R_0805_2012Metric_Pad1.15x1.40mm_HandSolder, F.Cu at (194.1, 154.4)
- added R2: 10K, Resistor_SMD:R_0805_2012Metric_Pad1.15x1.40mm_HandSolder, F.Cu at (41.7, 154.4)
- added R2: 10K, Resistor_SMD:R_0805_2012Metric_Pad1.15x1.40mm_HandSolder, F.Cu at (244.9, 80.7)
- added R2: 10K, Resistor_SMD:R_0805_2012Metric_Pad1.15x1.40mm_HandSolder, F.Cu at (194.1, 80.7)
- added R2: 10K, Resistor_SMD:R_0805_2012Metric_Pad1.15x1.40mm_HandSolder, F.Cu at (143.3, 80.7)
- added R2: 10K, Resistor_SMD:R_0805_2012Metric_Pad1.15x1.40mm_HandSolder, F.Cu at (92.5, 80.7)
- added R3: 10K, Resistor_SMD:R_0805_2012Metric_Pad1.15x1.40mm_HandSolder, F.Cu at (154.2, 140.0)
- added R3: 10K, Resistor_SMD:R_0805_2012Metric_Pad1.15x1.40mm_HandSolder, F.Cu at (52.6, 66.4)
- added R3: 10K, Resistor_SMD:R_0805_2012Metric_Pad1.15x1.40mm_HandSolder, F.Cu at (103.4, 140.0)
- added R3: 10K, Resistor_SMD:R_0805_2012Metric_Pad1.15x1.40mm_HandSolder, F.Cu at (255.8, 140.0)
- added R3: 10K, Resistor_SMD:R_0805_2012Metric_Pad1.15x1.40mm_HandSolder, F.Cu at (205.0, 140.0)
- added R3: 10K, Resistor_SMD:R_0805_2012Metric_Pad1.15x1.40mm_HandSolder, F.Cu at (52.6, 140.0)
- added R3: 10K, Resistor_SMD:R_0805_2012Metric_Pad1.15x1.40mm_HandSolder, F.Cu at (255.8, 66.4)
- added R3: 10K, Resistor_SMD:R_0805_2012Metric_Pad1.15x1.40mm_HandSolder, F.Cu at (205.0, 66.4)
- added R3: 10K, Resistor_SMD:R_0805_2012Metric_Pad1.15x1.40mm_HandSolder, F.Cu at (154.2, 66.4)
- added R3: 10K, Resistor_SMD:R_0805_2012Metric_Pad1.15x1.40mm_HandSolder, F.Cu at (103.4, 66.4)
- added R4: 10K, Resistor_SMD:R_0805_2012Metric_Pad1.15x1.40mm_HandSolder, F.Cu at (77.0, 140.1)
- added R4: 10K, Resistor_SMD:R_0805_2012Metric_Pad1.15x1.40mm_HandSolder, F.Cu at (26.2, 66.4)
- added R4: 10K, Resistor_SMD:R_0805_2012Metric_Pad1.15x1.40mm_HandSolder, F.Cu at (127.8, 140.1)
- added R4: 10K, Resistor_SMD:R_0805_2012Metric_Pad1.15x1.40mm_HandSolder, F.Cu at (178.6, 140.1)
- added R4: 10K, Resistor_SMD:R_0805_2012Metric_Pad1.15x1.40mm_HandSolder, F.Cu at (229.4, 140.1)
- added R4: 10K, Resistor_SMD:R_0805_2012Metric_Pad1.15x1.40mm_HandSolder, F.Cu at (26.2, 140.1)
- added R4: 10K, Resistor_SMD:R_0805_2012Metric_Pad1.15x1.40mm_HandSolder, F.Cu at (229.4, 66.4)
- added R4: 10K, Resistor_SMD:R_0805_2012Metric_Pad1.15x1.40mm_HandSolder, F.Cu at (178.6, 66.4)
- added R4: 10K, Resistor_SMD:R_0805_2012Metric_Pad1.15x1.40mm_HandSolder, F.Cu at (127.8, 66.4)
- added R4: 10K, Resistor_SMD:R_0805_2012Metric_Pad1.15x1.40mm_HandSolder, F.Cu at (77.0, 66.4)
- added U1: IRF7476, Package_SO:PowerIntegrations_SO-8, F.Cu at (135.3, 146.6)
- added U1: IRF7476, Package_SO:PowerIntegrations_SO-8, F.Cu at (33.7, 72.9)
- added U1: IRF7476, Package_SO:PowerIntegrations_SO-8, F.Cu at (186.1, 146.6)
- added U1: IRF7476, Package_SO:PowerIntegrations_SO-8, F.Cu at (84.5, 146.6)
- added U1: IRF7476, Package_SO:PowerIntegrations_SO-8, F.Cu at (236.9, 146.6)
- added U1: IRF7476, Package_SO:PowerIntegrations_SO-8, F.Cu at (33.7, 146.6)
- added U1: IRF7476, Package_SO:PowerIntegrations_SO-8, F.Cu at (236.9, 72.9)
- added U1: IRF7476, Package_SO:PowerIntegrations_SO-8, F.Cu at (186.1, 72.9)
- added U1: IRF7476, Package_SO:PowerIntegrations_SO-8, F.Cu at (135.3, 72.9)
- added U1: IRF7476, Package_SO:PowerIntegrations_SO-8, F.Cu at (84.5, 72.9)
- added U2: LM1117-1.8, Package_TO_SOT_SMD:SOT-223-3_TabPin2, F.Cu at (254.8, 155.3)
- added U2: LM1117-1.8, Package_TO_SOT_SMD:SOT-223-3_TabPin2, F.Cu at (51.6, 81.6)
- added U2: LM1117-1.8, Package_TO_SOT_SMD:SOT-223-3_TabPin2, F.Cu at (51.6, 155.3)
- added U2: LM1117-1.8, Package_TO_SOT_SMD:SOT-223-3_TabPin2, F.Cu at (102.4, 155.3)
- added U2: LM1117-1.8, Package_TO_SOT_SMD:SOT-223-3_TabPin2, F.Cu at (153.2, 155.3)
- added U2: LM1117-1.8, Package_TO_SOT_SMD:SOT-223-3_TabPin2, F.Cu at (204.0, 155.3)
- added U2: LM1117-1.8, Package_TO_SOT_SMD:SOT-223-3_TabPin2, F.Cu at (254.8, 81.6)
- added U2: LM1117-1.8, Package_TO_SOT_SMD:SOT-223-3_TabPin2, F.Cu at (204.0, 81.6)
- added U2: LM1117-1.8, Package_TO_SOT_SMD:SOT-223-3_TabPin2, F.Cu at (153.2, 81.6)
- added U2: LM1117-1.8, Package_TO_SOT_SMD:SOT-223-3_TabPin2, F.Cu at (102.4, 81.6)
- added U3: IRF7476, Package_SO:PowerIntegrations_SO-8, F.Cu at (101.7, 146.1)
- added U3: IRF7476, Package_SO:PowerIntegrations_SO-8, F.Cu at (50.9, 72.5)
- added U3: IRF7476, Package_SO:PowerIntegrations_SO-8, F.Cu at (203.3, 146.1)
- added U3: IRF7476, Package_SO:PowerIntegrations_SO-8, F.Cu at (152.5, 146.1)
- added U3: IRF7476, Package_SO:PowerIntegrations_SO-8, F.Cu at (254.1, 146.1)
- added U3: IRF7476, Package_SO:PowerIntegrations_SO-8, F.Cu at (50.9, 146.1)
- added U3: IRF7476, Package_SO:PowerIntegrations_SO-8, F.Cu at (254.1, 72.5)
- added U3: IRF7476, Package_SO:PowerIntegrations_SO-8, F.Cu at (203.3, 72.5)
- added U3: IRF7476, Package_SO:PowerIntegrations_SO-8, F.Cu at (152.5, 72.5)
- added U3: IRF7476, Package_SO:PowerIntegrations_SO-8, F.Cu at (101.7, 72.5)
- added U4: IRF7476, Package_SO:PowerIntegrations_SO-8, F.Cu at (126.1, 146.6)
- added U4: IRF7476, Package_SO:PowerIntegrations_SO-8, F.Cu at (24.5, 72.9)
- added U4: IRF7476, Package_SO:PowerIntegrations_SO-8, F.Cu at (227.7, 146.6)
- added U4: IRF7476, Package_SO:PowerIntegrations_SO-8, F.Cu at (75.3, 146.6)
- added U4: IRF7476, Package_SO:PowerIntegrations_SO-8, F.Cu at (176.9, 146.6)
- added U4: IRF7476, Package_SO:PowerIntegrations_SO-8, F.Cu at (24.5, 146.6)
- added U4: IRF7476, Package_SO:PowerIntegrations_SO-8, F.Cu at (227.7, 72.9)
- added U4: IRF7476, Package_SO:PowerIntegrations_SO-8, F.Cu at (176.9, 72.9)
- added U4: IRF7476, Package_SO:PowerIntegrations_SO-8, F.Cu at (126.1, 72.9)
- added U4: IRF7476, Package_SO:PowerIntegrations_SO-8, F.Cu at (75.3, 72.9)
Routing:
- net (no net): track 76.7 -> 3658.2 mm
- net GND: track 0.00 -> 96.8 mm
- net +5V: track 0.00 -> 88.1 mm
- net +1V8: track 0.00 -> 70.4 mm
- net /SCK: track 0.00 -> 32.2 mm
- net Net-(J3-Pad6): track 0.00 -> 29.5 mm
- net /MISO: track 0.00 -> 17.2 mm
- net Net-(J3-Pad2): track 0.00 -> 16.0 mm
- net /CS: track 0.00 -> 15.4 mm
- net Net-(J3-Pad3): track 0.00 -> 15.3 mm
- net Net-(J1-Pad1): track 15.1 -> 0.00 mm
- net /MOSI: track 0.00 -> 14.5 mm
- net Net-(D1-Pad1): track 0.00 -> 11.0 mm
- net Net-(J1-Pad2): track 6.37 -> 0.00 mm
- net Net-(J1-Pad3): track 4.14 -> 0.00 mm
- added copper zone on F.Cu, net (none)
- added copper zone on F.Cu, net GND
Other:
- board text added: "by KK"

Commit message: Konwerter update
-> Poprawiony schemat konwertera
-> Samodzielna płytka z konwerterem
-> poprawiony symbol karty aby pasował do footprintu
Parts:
- removed the C1 at (210.1, 157.9)
- removed the C1 at (57.7, 84.2)
- removed the C1 at (260.9, 157.9)
- removed the C1 at (57.7, 157.9)
- removed the C1 at (108.5, 157.9)
- removed the C1 at (159.3, 157.9)
- removed the C1 at (260.9, 84.2)
- removed the C1 at (210.1, 84.2)
- removed the C1 at (159.3, 84.2)
- removed the C1 at (108.5, 84.2)
- removed the C2 at (57.9, 148.3)
- removed the C2 at (57.9, 74.6)
- removed the C2 at (261.1, 148.3)
- removed the C2 at (210.3, 148.3)
- removed the C2 at (159.5, 148.3)
- removed the C2 at (108.7, 148.3)
- removed the C2 at (261.1, 74.6)
- removed the C2 at (210.3, 74.6)
- removed the C2 at (159.5, 74.6)
- removed the C2 at (108.7, 74.6)
- removed D1 (x10): 4,7V, Diode_THT:D_DO-41_SOD81_P7.62mm_Horizontal
- removed the J1 at (73.1, 154.5)
- removed the J1 at (22.3, 80.9)
- removed the J1 at (123.9, 154.5)
- removed the J1 at (174.7, 154.5)
- removed the J1 at (225.5, 154.5)
- removed the J1 at (22.3, 154.5)
- removed the J1 at (225.5, 80.9)
- removed the J1 at (174.7, 80.9)
- removed the J1 at (123.9, 80.9)
- removed the J1 at (73.1, 80.9)
- removed J3 (x10): Micro_SD_Card, Connector_Card:SD_Kyocera_145638009511859+
- removed the R1 at (139.1, 140.6)
- removed the R1 at (37.5, 66.9)
- removed the R1 at (189.9, 140.6)
- removed the R1 at (240.7, 140.6)
- removed the R1 at (88.3, 140.6)
- removed the R1 at (37.5, 140.6)
- removed the R1 at (240.7, 66.9)
- removed the R1 at (189.9, 66.9)
- removed the R1 at (139.1, 66.9)
- removed the R1 at (88.3, 66.9)
- removed the R2 at (92.5, 154.4)
- removed the R2 at (41.7, 80.7)
- removed the R2 at (244.9, 154.4)
- removed the R2 at (143.3, 154.4)
- removed the R2 at (194.1, 154.4)
- removed the R2 at (41.7, 154.4)
- removed the R2 at (244.9, 80.7)
- removed the R2 at (194.1, 80.7)
- removed the R2 at (143.3, 80.7)
- removed the R2 at (92.5, 80.7)
- removed the R3 at (154.2, 140.0)
- removed the R3 at (52.6, 66.4)
- removed the R3 at (103.4, 140.0)
- removed the R3 at (255.8, 140.0)
- removed the R3 at (205.0, 140.0)
- removed the R3 at (52.6, 140.0)
- removed the R3 at (255.8, 66.4)
- removed the R3 at (205.0, 66.4)
- removed the R3 at (154.2, 66.4)
- removed the R3 at (103.4, 66.4)
- removed the R4 at (77.0, 140.1)
- removed the R4 at (26.2, 66.4)
- removed the R4 at (127.8, 140.1)
- removed the R4 at (178.6, 140.1)
- removed the R4 at (229.4, 140.1)
- removed the R4 at (26.2, 140.1)
- removed the R4 at (229.4, 66.4)
- removed the R4 at (178.6, 66.4)
- removed the R4 at (127.8, 66.4)
- removed the R4 at (77.0, 66.4)
- removed the U1 at (135.3, 146.6)
- removed the U1 at (33.7, 72.9)
- removed the U1 at (186.1, 146.6)
- removed the U1 at (84.5, 146.6)
- removed the U1 at (236.9, 146.6)
- removed the U1 at (33.7, 146.6)
- removed the U1 at (236.9, 72.9)
- removed the U1 at (186.1, 72.9)
- removed the U1 at (135.3, 72.9)
- removed the U1 at (84.5, 72.9)
- removed the U2 at (254.8, 155.3)
- removed the U2 at (51.6, 81.6)
- removed the U2 at (51.6, 155.3)
- removed the U2 at (102.4, 155.3)
- removed the U2 at (153.2, 155.3)
- removed the U2 at (204.0, 155.3)
- removed the U2 at (254.8, 81.6)
- removed the U2 at (204.0, 81.6)
- removed the U2 at (153.2, 81.6)
- removed the U2 at (102.4, 81.6)
- removed the U3 at (101.7, 146.1)
- removed the U3 at (50.9, 72.5)
- removed the U3 at (203.3, 146.1)
- removed the U3 at (152.5, 146.1)
- removed the U3 at (254.1, 146.1)
- removed the U3 at (50.9, 146.1)
- removed the U3 at (254.1, 72.5)
- removed the U3 at (203.3, 72.5)
- removed the U3 at (152.5, 72.5)
- removed the U3 at (101.7, 72.5)
- removed the U4 at (126.1, 146.6)
- removed the U4 at (24.5, 72.9)
- removed the U4 at (227.7, 146.6)
- removed the U4 at (75.3, 146.6)
- removed the U4 at (176.9, 146.6)
- removed the U4 at (24.5, 146.6)
- removed the U4 at (227.7, 72.9)
- removed the U4 at (176.9, 72.9)
- removed the U4 at (126.1, 72.9)
- removed the U4 at (75.3, 72.9)
- added C1: 100N, Connector_PinHeader_2.54mm:PinHeader_1x02_P2.54mm_Vertical, B.Cu at (74.9, 176.5)
- added C1: 100N, Connector_PinHeader_2.54mm:PinHeader_1x02_P2.54mm_Vertical, B.Cu at (181.6, 142.2)
- added C1: 100N, Connector_PinHeader_2.54mm:PinHeader_1x02_P2.54mm_Vertical, B.Cu at (146.1, 142.2)
- added C1: 100N, Connector_PinHeader_2.54mm:PinHeader_1x02_P2.54mm_Vertical, B.Cu at (110.5, 142.2)
- added C1: 100N, Connector_PinHeader_2.54mm:PinHeader_1x02_P2.54mm_Vertical, B.Cu at (217.2, 142.2)
- added C1: 100N, Connector_PinHeader_2.54mm:PinHeader_1x02_P2.54mm_Vertical, B.Cu at (39.4, 142.2)
- added C1: 100N, Connector_PinHeader_2.54mm:PinHeader_1x02_P2.54mm_Vertical, B.Cu at (74.9, 108.0)
- added C1: 100N, Connector_PinHeader_2.54mm:PinHeader_1x02_P2.54mm_Vertical, B.Cu at (252.7, 108.0)
- added C1: 100N, Connector_PinHeader_2.54mm:PinHeader_1x02_P2.54mm_Vertical, B.Cu at (181.6, 108.0)
- added C1: 100N, Connector_PinHeader_2.54mm:PinHeader_1x02_P2.54mm_Vertical, B.Cu at (146.1, 108.0)
- added C1: 100N, Connector_PinHeader_2.54mm:PinHeader_1x02_P2.54mm_Vertical, B.Cu at (110.5, 108.0)
- added C1: 100N, Connector_PinHeader_2.54mm:PinHeader_1x02_P2.54mm_Vertical, B.Cu at (252.7, 176.5)
- added C1: 100N, Connector_PinHeader_2.54mm:PinHeader_1x02_P2.54mm_Vertical, B.Cu at (217.2, 108.0)
- added C1: 100N, Connector_PinHeader_2.54mm:PinHeader_1x02_P2.54mm_Vertical, B.Cu at (39.4, 108.0)
- added C1: 100N, Connector_PinHeader_2.54mm:PinHeader_1x02_P2.54mm_Vertical, B.Cu at (74.9, 73.7)
- added C1: 100N, Connector_PinHeader_2.54mm:PinHeader_1x02_P2.54mm_Vertical, B.Cu at (252.7, 73.7)
- added C1: 100N, Connector_PinHeader_2.54mm:PinHeader_1x02_P2.54mm_Vertical, B.Cu at (181.6, 73.7)
- added C1: 100N, Connector_PinHeader_2.54mm:PinHeader_1x02_P2.54mm_Vertical, B.Cu at (146.1, 73.7)
- added C1: 100N, Connector_PinHeader_2.54mm:PinHeader_1x02_P2.54mm_Vertical, B.Cu at (110.5, 73.7)
- added C1: 100N, Connector_PinHeader_2.54mm:PinHeader_1x02_P2.54mm_Vertical, B.Cu at (217.2, 73.7)
- added C1: 100N, Connector_PinHeader_2.54mm:PinHeader_1x02_P2.54mm_Vertical, B.Cu at (39.4, 73.7)
- added C1: 100N, Connector_PinHeader_2.54mm:PinHeader_1x02_P2.54mm_Vertical, B.Cu at (252.7, 39.4)
- added C1: 100N, Connector_PinHeader_2.54mm:PinHeader_1x02_P2.54mm_Vertical, B.Cu at (181.6, 176.5)
- added C1: 100N, Connector_PinHeader_2.54mm:PinHeader_1x02_P2.54mm_Vertical, B.Cu at (217.2, 39.4)
- added C1: 100N, Connector_PinHeader_2.54mm:PinHeader_1x02_P2.54mm_Vertical, B.Cu at (181.6, 39.4)
- added C1: 100N, Connector_PinHeader_2.54mm:PinHeader_1x02_P2.54mm_Vertical, B.Cu at (146.1, 39.4)
- added C1: 100N, Connector_PinHeader_2.54mm:PinHeader_1x02_P2.54mm_Vertical, B.Cu at (110.5, 39.4)
- added C1: 100N, Connector_PinHeader_2.54mm:PinHeader_1x02_P2.54mm_Vertical, B.Cu at (74.9, 39.4)
- added C1: 100N, Connector_PinHeader_2.54mm:PinHeader_1x02_P2.54mm_Vertical, B.Cu at (39.4, 39.4)
- added C1: 100N, Connector_PinHeader_2.54mm:PinHeader_1x02_P2.54mm_Vertical, B.Cu at (146.1, 176.5)
- added C1: 100N, Connector_PinHeader_2.54mm:PinHeader_1x02_P2.54mm_Vertical, B.Cu at (110.5, 176.5)
- added C1: 100N, Connector_PinHeader_2.54mm:PinHeader_1x02_P2.54mm_Vertical, B.Cu at (217.2, 176.5)
- added C1: 100N, Connector_PinHeader_2.54mm:PinHeader_1x02_P2.54mm_Vertical, B.Cu at (39.4, 176.5)
- added C1: 100N, Connector_PinHeader_2.54mm:PinHeader_1x02_P2.54mm_Vertical, B.Cu at (74.9, 142.2)
- added C1: 100N, Connector_PinHeader_2.54mm:PinHeader_1x02_P2.54mm_Vertical, B.Cu at (252.7, 142.2)
- added C2: 100N, Connector_PinHeader_2.54mm:PinHeader_1x02_P2.54mm_Vertical, B.Cu at (58.4, 176.5)
- added C2: 100N, Connector_PinHeader_2.54mm:PinHeader_1x02_P2.54mm_Vertical, B.Cu at (94.0, 142.2)
- added C2: 100N, Connector_PinHeader_2.54mm:PinHeader_1x02_P2.54mm_Vertical, B.Cu at (236.2, 142.2)
- added C2: 100N, Connector_PinHeader_2.54mm:PinHeader_1x02_P2.54mm_Vertical, B.Cu at (200.7, 142.2)
- added C2: 100N, Connector_PinHeader_2.54mm:PinHeader_1x02_P2.54mm_Vertical, B.Cu at (165.1, 142.2)
- added C2: 100N, Connector_PinHeader_2.54mm:PinHeader_1x02_P2.54mm_Vertical, B.Cu at (129.5, 142.2)
- added C2: 100N, Connector_PinHeader_2.54mm:PinHeader_1x02_P2.54mm_Vertical, B.Cu at (58.4, 108.0)
- added C2: 100N, Connector_PinHeader_2.54mm:PinHeader_1x02_P2.54mm_Vertical, B.Cu at (22.9, 108.0)
- added C2: 100N, Connector_PinHeader_2.54mm:PinHeader_1x02_P2.54mm_Vertical, B.Cu at (94.0, 108.0)
- added C2: 100N, Connector_PinHeader_2.54mm:PinHeader_1x02_P2.54mm_Vertical, B.Cu at (236.2, 108.0)
- added C2: 100N, Connector_PinHeader_2.54mm:PinHeader_1x02_P2.54mm_Vertical, B.Cu at (200.7, 108.0)
- added C2: 100N, Connector_PinHeader_2.54mm:PinHeader_1x02_P2.54mm_Vertical, B.Cu at (22.9, 176.5)
- added C2: 100N, Connector_PinHeader_2.54mm:PinHeader_1x02_P2.54mm_Vertical, B.Cu at (165.1, 108.0)
- added C2: 100N, Connector_PinHeader_2.54mm:PinHeader_1x02_P2.54mm_Vertical, B.Cu at (129.5, 108.0)
- added C2: 100N, Connector_PinHeader_2.54mm:PinHeader_1x02_P2.54mm_Vertical, B.Cu at (58.4, 73.7)
- added C2: 100N, Connector_PinHeader_2.54mm:PinHeader_1x02_P2.54mm_Vertical, B.Cu at (22.9, 73.7)
- added C2: 100N, Connector_PinHeader_2.54mm:PinHeader_1x02_P2.54mm_Vertical, B.Cu at (94.0, 73.7)
- added C2: 100N, Connector_PinHeader_2.54mm:PinHeader_1x02_P2.54mm_Vertical, B.Cu at (236.2, 73.7)
- added C2: 100N, Connector_PinHeader_2.54mm:PinHeader_1x02_P2.54mm_Vertical, B.Cu at (200.7, 73.7)
- added C2: 100N, Connector_PinHeader_2.54mm:PinHeader_1x02_P2.54mm_Vertical, B.Cu at (165.1, 73.7)
- added C2: 100N, Connector_PinHeader_2.54mm:PinHeader_1x02_P2.54mm_Vertical, B.Cu at (129.5, 73.7)
- added C2: 100N, Connector_PinHeader_2.54mm:PinHeader_1x02_P2.54mm_Vertical, B.Cu at (236.2, 39.4)
- added C2: 100N, Connector_PinHeader_2.54mm:PinHeader_1x02_P2.54mm_Vertical, B.Cu at (94.0, 176.5)
- added C2: 100N, Connector_PinHeader_2.54mm:PinHeader_1x02_P2.54mm_Vertical, B.Cu at (200.7, 39.4)
- added C2: 100N, Connector_PinHeader_2.54mm:PinHeader_1x02_P2.54mm_Vertical, B.Cu at (165.1, 39.4)
- added C2: 100N, Connector_PinHeader_2.54mm:PinHeader_1x02_P2.54mm_Vertical, B.Cu at (129.5, 39.4)
- added C2: 100N, Connector_PinHeader_2.54mm:PinHeader_1x02_P2.54mm_Vertical, B.Cu at (94.0, 39.4)
- added C2: 100N, Connector_PinHeader_2.54mm:PinHeader_1x02_P2.54mm_Vertical, B.Cu at (58.4, 39.4)
- added C2: 100N, Connector_PinHeader_2.54mm:PinHeader_1x02_P2.54mm_Vertical, B.Cu at (22.9, 39.4)
- added C2: 100N, Connector_PinHeader_2.54mm:PinHeader_1x02_P2.54mm_Vertical, B.Cu at (236.2, 176.5)
- added C2: 100N, Connector_PinHeader_2.54mm:PinHeader_1x02_P2.54mm_Vertical, B.Cu at (200.7, 176.5)
- added C2: 100N, Connector_PinHeader_2.54mm:PinHeader_1x02_P2.54mm_Vertical, B.Cu at (165.1, 176.5)
- added C2: 100N, Connector_PinHeader_2.54mm:PinHeader_1x02_P2.54mm_Vertical, B.Cu at (129.5, 176.5)
- added C2: 100N, Connector_PinHeader_2.54mm:PinHeader_1x02_P2.54mm_Vertical, B.Cu at (58.4, 142.2)
- added C2: 100N, Connector_PinHeader_2.54mm:PinHeader_1x02_P2.54mm_Vertical, B.Cu at (22.9, 142.2)
- added J1: Conn_01x06_Male, Connector_PinHeader_2.54mm:PinHeader_1x06_P2.54mm_Vertical, B.Cu at (229.7, 167.6)
- added J1: Conn_01x06_Male, Connector_PinHeader_2.54mm:PinHeader_1x06_P2.54mm_Vertical, B.Cu at (123.0, 133.3)
- added J1: Conn_01x06_Male, Connector_PinHeader_2.54mm:PinHeader_1x06_P2.54mm_Vertical, B.Cu at (87.4, 133.3)
- added J1: Conn_01x06_Male, Connector_PinHeader_2.54mm:PinHeader_1x06_P2.54mm_Vertical, B.Cu at (51.9, 133.3)
- added J1: Conn_01x06_Male, Connector_PinHeader_2.54mm:PinHeader_1x06_P2.54mm_Vertical, B.Cu at (194.1, 133.3)
- added J1: Conn_01x06_Male, Connector_PinHeader_2.54mm:PinHeader_1x06_P2.54mm_Vertical, B.Cu at (16.3, 133.3)
- added J1: Conn_01x06_Male, Connector_PinHeader_2.54mm:PinHeader_1x06_P2.54mm_Vertical, B.Cu at (229.7, 99.1)
- added J1: Conn_01x06_Male, Connector_PinHeader_2.54mm:PinHeader_1x06_P2.54mm_Vertical, B.Cu at (158.5, 99.1)
- added J1: Conn_01x06_Male, Connector_PinHeader_2.54mm:PinHeader_1x06_P2.54mm_Vertical, B.Cu at (123.0, 99.1)
- added J1: Conn_01x06_Male, Connector_PinHeader_2.54mm:PinHeader_1x06_P2.54mm_Vertical, B.Cu at (87.4, 99.1)
- added J1: Conn_01x06_Male, Connector_PinHeader_2.54mm:PinHeader_1x06_P2.54mm_Vertical, B.Cu at (51.9, 99.1)
- added J1: Conn_01x06_Male, Connector_PinHeader_2.54mm:PinHeader_1x06_P2.54mm_Vertical, B.Cu at (158.5, 167.6)
- added J1: Conn_01x06_Male, Connector_PinHeader_2.54mm:PinHeader_1x06_P2.54mm_Vertical, B.Cu at (194.1, 99.1)
- added J1: Conn_01x06_Male, Connector_PinHeader_2.54mm:PinHeader_1x06_P2.54mm_Vertical, B.Cu at (16.3, 99.1)
- added J1: Conn_01x06_Male, Connector_PinHeader_2.54mm:PinHeader_1x06_P2.54mm_Vertical, B.Cu at (229.7, 64.8)
- added J1: Conn_01x06_Male, Connector_PinHeader_2.54mm:PinHeader_1x06_P2.54mm_Vertical, B.Cu at (158.5, 64.8)
- added J1: Conn_01x06_Male, Connector_PinHeader_2.54mm:PinHeader_1x06_P2.54mm_Vertical, B.Cu at (123.0, 64.8)
- added J1: Conn_01x06_Male, Connector_PinHeader_2.54mm:PinHeader_1x06_P2.54mm_Vertical, B.Cu at (87.4, 64.8)
- added J1: Conn_01x06_Male, Connector_PinHeader_2.54mm:PinHeader_1x06_P2.54mm_Vertical, B.Cu at (51.9, 64.8)
- added J1: Conn_01x06_Male, Connector_PinHeader_2.54mm:PinHeader_1x06_P2.54mm_Vertical, B.Cu at (194.1, 64.8)
- added J1: Conn_01x06_Male, Connector_PinHeader_2.54mm:PinHeader_1x06_P2.54mm_Vertical, B.Cu at (16.3, 64.8)
- added J1: Conn_01x06_Male, Connector_PinHeader_2.54mm:PinHeader_1x06_P2.54mm_Vertical, B.Cu at (229.7, 30.5)
- added J1: Conn_01x06_Male, Connector_PinHeader_2.54mm:PinHeader_1x06_P2.54mm_Vertical, B.Cu at (123.0, 167.6)
- added J1: Conn_01x06_Male, Connector_PinHeader_2.54mm:PinHeader_1x06_P2.54mm_Vertical, B.Cu at (194.1, 30.5)
- added J1: Conn_01x06_Male, Connector_PinHeader_2.54mm:PinHeader_1x06_P2.54mm_Vertical, B.Cu at (158.5, 30.5)
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Routing:
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Other:
- board text added: "Master"
- board text added: "Slave"
- board text removed: "by KK"

Commit message: Dodano "by KK"
Parts:
- removed the C1 at (74.9, 176.5)
- removed the C1 at (181.6, 142.2)
- removed the C1 at (146.1, 142.2)
- removed the C1 at (110.5, 142.2)
- removed the C1 at (217.2, 142.2)
- removed the C1 at (74.9, 108.0)
- removed the C1 at (252.7, 108.0)
- removed the C1 at (181.6, 108.0)
- removed the C1 at (146.1, 108.0)
- removed the C1 at (110.5, 108.0)
- removed the C1 at (252.7, 176.5)
- removed the C1 at (217.2, 108.0)
- removed the C1 at (74.9, 73.7)
- removed the C1 at (252.7, 73.7)
- removed the C1 at (181.6, 73.7)
- removed the C1 at (146.1, 73.7)
- removed the C1 at (110.5, 73.7)
- removed the C1 at (217.2, 73.7)
- removed the C1 at (252.7, 39.4)
- removed the C1 at (181.6, 176.5)
- removed the C1 at (217.2, 39.4)
- removed the C1 at (181.6, 39.4)
- removed the C1 at (146.1, 39.4)
- removed the C1 at (110.5, 39.4)
- removed the C1 at (74.9, 39.4)
- removed the C1 at (146.1, 176.5)
- removed the C1 at (110.5, 176.5)
- removed the C1 at (217.2, 176.5)
- removed the C1 at (74.9, 142.2)
- removed the C1 at (252.7, 142.2)
- removed the C2 at (58.4, 176.5)
- removed the C2 at (94.0, 142.2)
- removed the C2 at (236.2, 142.2)
- removed the C2 at (200.7, 142.2)
- removed the C2 at (165.1, 142.2)
- removed the C2 at (129.5, 142.2)
- removed the C2 at (58.4, 108.0)
- removed the C2 at (94.0, 108.0)
- removed the C2 at (236.2, 108.0)
- removed the C2 at (200.7, 108.0)
- removed the C2 at (165.1, 108.0)
- removed the C2 at (129.5, 108.0)
- removed the C2 at (58.4, 73.7)
- removed the C2 at (94.0, 73.7)
- removed the C2 at (236.2, 73.7)
- removed the C2 at (200.7, 73.7)
- removed the C2 at (165.1, 73.7)
- removed the C2 at (129.5, 73.7)
- removed the C2 at (236.2, 39.4)
- removed the C2 at (94.0, 176.5)
- removed the C2 at (200.7, 39.4)
- removed the C2 at (165.1, 39.4)
- removed the C2 at (129.5, 39.4)
- removed the C2 at (94.0, 39.4)
- removed the C2 at (58.4, 39.4)
- removed the C2 at (236.2, 176.5)
- removed the C2 at (200.7, 176.5)
- removed the C2 at (165.1, 176.5)
- removed the C2 at (129.5, 176.5)
- removed the C2 at (58.4, 142.2)
- removed the J1 at (229.7, 167.6)
- removed the J1 at (123.0, 133.3)
- removed the J1 at (87.4, 133.3)
- removed the J1 at (51.9, 133.3)
- removed the J1 at (194.1, 133.3)
- removed the J1 at (229.7, 99.1)
- removed the J1 at (158.5, 99.1)
- removed the J1 at (123.0, 99.1)
- removed the J1 at (87.4, 99.1)
- removed the J1 at (51.9, 99.1)
- removed the J1 at (158.5, 167.6)
- removed the J1 at (194.1, 99.1)
- removed the J1 at (229.7, 64.8)
- removed the J1 at (158.5, 64.8)
- removed the J1 at (123.0, 64.8)
- removed the J1 at (87.4, 64.8)
- removed the J1 at (51.9, 64.8)
- removed the J1 at (194.1, 64.8)
- removed the J1 at (229.7, 30.5)
- removed the J1 at (123.0, 167.6)
- removed the J1 at (194.1, 30.5)
- removed the J1 at (158.5, 30.5)
- removed the J1 at (123.0, 30.5)
- removed the J1 at (87.4, 30.5)
- removed the J1 at (51.9, 30.5)
- removed the J1 at (87.4, 167.6)
- removed the J1 at (51.9, 167.6)
- removed the J1 at (194.1, 167.6)
- removed the J1 at (229.7, 133.3)
- removed the J1 at (158.5, 133.3)
- removed the J2 at (77.2, 167.6)
- removed the J2 at (183.9, 133.3)
- removed the J2 at (255.0, 133.3)
- removed the J2 at (148.3, 133.3)
- removed the J2 at (112.8, 133.3)
- removed the J2 at (219.5, 133.3)
- removed the J2 at (77.2, 99.1)
- removed the J2 at (183.9, 99.1)
- removed the J2 at (255.0, 99.1)
- removed the J2 at (148.3, 99.1)
- removed the J2 at (112.8, 99.1)
- removed the J2 at (219.5, 99.1)
- removed the J2 at (77.2, 64.8)
- removed the J2 at (183.9, 64.8)
- removed the J2 at (255.0, 64.8)
- removed the J2 at (148.3, 64.8)
- removed the J2 at (112.8, 64.8)
- removed the J2 at (219.5, 64.8)
- removed the J2 at (255.0, 30.5)
- removed the J2 at (183.9, 167.6)
- removed the J2 at (219.5, 30.5)
- removed the J2 at (183.9, 30.5)
- removed the J2 at (148.3, 30.5)
- removed the J2 at (112.8, 30.5)
- removed the J2 at (77.2, 30.5)
- removed the J2 at (255.0, 167.6)
- removed the J2 at (148.3, 167.6)
- removed the J2 at (112.8, 167.6)
- removed the J2 at (219.5, 167.6)
- removed the J2 at (77.2, 133.3)
- removed the R1 at (72.4, 171.4)
- removed the R1 at (179.1, 137.2)
- removed the R1 at (214.6, 137.2)
- removed the R1 at (143.5, 137.2)
- removed the R1 at (108.0, 137.2)
- removed the R1 at (72.4, 102.9)
- removed the R1 at (250.2, 102.9)
- removed the R1 at (179.1, 102.9)
- removed the R1 at (214.6, 102.9)
- removed the R1 at (143.5, 102.9)
- removed the R1 at (250.2, 171.4)
- removed the R1 at (108.0, 102.9)
- removed the R1 at (72.4, 68.6)
- removed the R1 at (250.2, 68.6)
- removed the R1 at (179.1, 68.6)
- removed the R1 at (214.6, 68.6)
- removed the R1 at (143.5, 68.6)
- removed the R1 at (108.0, 68.6)
- removed the R1 at (250.2, 34.3)
- removed the R1 at (179.1, 171.4)
- removed the R1 at (214.6, 34.3)
- removed the R1 at (179.1, 34.3)
- removed the R1 at (143.5, 34.3)
- removed the R1 at (108.0, 34.3)
- removed the R1 at (72.4, 34.3)
- removed the R1 at (214.6, 171.4)
- removed the R1 at (143.5, 171.4)
- removed the R1 at (108.0, 171.4)
- removed the R1 at (72.4, 137.2)
- removed the R1 at (250.2, 137.2)
- removed the R2 at (57.1, 153.7)
- removed the R2 at (163.8, 119.4)
- removed the R2 at (199.4, 119.4)
- removed the R2 at (128.3, 119.4)
- removed the R2 at (92.7, 119.4)
- removed the R2 at (57.1, 85.1)
- removed the R2 at (234.9, 85.1)
- removed the R2 at (163.8, 85.1)
- removed the R2 at (199.4, 85.1)
- removed the R2 at (234.9, 153.7)
- removed the R2 at (128.3, 85.1)
- removed the R2 at (92.7, 85.1)
- removed the R2 at (57.1, 50.8)
- removed the R2 at (234.9, 50.8)
- removed the R2 at (163.8, 50.8)
- removed the R2 at (199.4, 50.8)
- removed the R2 at (128.3, 50.8)
- removed the R2 at (92.7, 50.8)
- removed the R2 at (234.9, 16.5)
- removed the R2 at (163.8, 153.7)
- removed the R2 at (199.4, 16.5)
- removed the R2 at (163.8, 16.5)
- removed the R2 at (128.3, 16.5)
- removed the R2 at (92.7, 16.5)
- removed the R2 at (57.1, 16.5)
- removed the R2 at (199.4, 153.7)
- removed the R2 at (128.3, 153.7)
- removed the R2 at (92.7, 153.7)
- removed the R2 at (57.1, 119.4)
- removed the R2 at (234.9, 119.4)
- removed the R3 at (177.3, 119.4)
- removed the R3 at (212.9, 119.4)
- removed the R3 at (248.4, 119.4)
- removed the R3 at (70.6, 119.4)
- removed the R3 at (106.2, 119.4)
- removed the R3 at (141.7, 85.1)
- removed the R3 at (177.3, 85.1)
- removed the R3 at (212.9, 85.1)
- removed the R3 at (248.4, 85.1)
- removed the R3 at (141.7, 153.7)
- removed the R3 at (70.6, 85.1)
- removed the R3 at (106.2, 85.1)
- removed the R3 at (141.7, 50.8)
- removed the R3 at (177.3, 50.8)
- removed the R3 at (212.9, 50.8)
- removed the R3 at (248.4, 50.8)
- removed the R3 at (70.6, 50.8)
- removed the R3 at (106.2, 50.8)
- removed the R3 at (248.4, 16.5)
- removed the R3 at (177.3, 153.7)
- removed the R3 at (212.9, 16.5)
- removed the R3 at (177.3, 16.5)
- removed the R3 at (141.7, 16.5)
- removed the R3 at (106.2, 16.5)
- removed the R3 at (70.6, 16.5)
- removed the R3 at (212.9, 153.7)
- removed the R3 at (248.4, 153.7)
- removed the R3 at (70.6, 153.7)
- removed the R3 at (106.2, 153.7)
- removed the R3 at (141.7, 119.4)
- removed the R4 at (200.7, 137.2)
- removed the R4 at (58.4, 137.2)
- removed the R4 at (94.0, 137.2)
- removed the R4 at (129.5, 137.2)
- removed the R4 at (165.1, 137.2)
- removed the R4 at (236.2, 102.9)
- removed the R4 at (200.7, 102.9)
- removed the R4 at (58.4, 102.9)
- removed the R4 at (94.0, 102.9)
- removed the R4 at (236.2, 171.4)
- removed the R4 at (129.5, 102.9)
- removed the R4 at (165.1, 102.9)
- removed the R4 at (236.2, 68.6)
- removed the R4 at (200.7, 68.6)
- removed the R4 at (58.4, 68.6)
- removed the R4 at (94.0, 68.6)
- removed the R4 at (129.5, 68.6)
- removed the R4 at (165.1, 68.6)
- removed the R4 at (236.2, 34.3)
- removed the R4 at (200.7, 171.4)
- removed the R4 at (200.7, 34.3)
- removed the R4 at (165.1, 34.3)
- removed the R4 at (129.5, 34.3)
- removed the R4 at (94.0, 34.3)
- removed the R4 at (58.4, 34.3)
- removed the R4 at (58.4, 171.4)
- removed the R4 at (94.0, 171.4)
- removed the R4 at (129.5, 171.4)
- removed the R4 at (165.1, 171.4)
- removed the R4 at (236.2, 137.2)
- removed the U1 at (69.1, 166.4)
- removed the U1 at (211.3, 132.1)
- removed the U1 at (140.2, 132.1)
- removed the U1 at (175.8, 132.1)
- removed the U1 at (104.6, 132.1)
- removed the U1 at (69.1, 97.8)
- removed the U1 at (246.9, 97.8)
- removed the U1 at (211.3, 97.8)
- removed the U1 at (140.2, 97.8)
- removed the U1 at (246.9, 166.4)
- removed the U1 at (175.8, 97.8)
- removed the U1 at (104.6, 97.8)
- removed the U1 at (69.1, 63.5)
- removed the U1 at (246.9, 63.5)
- removed the U1 at (211.3, 63.5)
- removed the U1 at (140.2, 63.5)
- removed the U1 at (175.8, 63.5)
- removed the U1 at (104.6, 63.5)
- removed the U1 at (246.9, 29.2)
- removed the U1 at (211.3, 166.4)
- removed the U1 at (211.3, 29.2)
- removed the U1 at (175.8, 29.2)
- removed the U1 at (140.2, 29.2)
- removed the U1 at (104.6, 29.2)
- removed the U1 at (69.1, 29.2)
- removed the U1 at (140.2, 166.4)
- removed the U1 at (175.8, 166.4)
- removed the U1 at (104.6, 166.4)
- removed the U1 at (69.1, 132.1)
- removed the U1 at (246.9, 132.1)
- removed the U2 at (207.0, 139.7)
- removed the U2 at (242.6, 139.7)
- removed the U2 at (135.9, 139.7)
- removed the U2 at (100.3, 139.7)
- removed the U2 at (64.8, 139.7)
- removed the U2 at (171.4, 105.4)
- removed the U2 at (207.0, 105.4)
- removed the U2 at (242.6, 105.4)
- removed the U2 at (135.9, 105.4)
- removed the U2 at (171.4, 174.0)
- removed the U2 at (100.3, 105.4)
- removed the U2 at (64.8, 105.4)
- removed the U2 at (171.4, 71.1)
- removed the U2 at (207.0, 71.1)
- removed the U2 at (242.6, 71.1)
- removed the U2 at (135.9, 71.1)
- removed the U2 at (100.3, 71.1)
- removed the U2 at (64.8, 71.1)
- removed the U2 at (242.6, 36.8)
- removed the U2 at (207.0, 174.0)
- removed the U2 at (207.0, 36.8)
- removed the U2 at (171.4, 36.8)
- removed the U2 at (135.9, 36.8)
- removed the U2 at (100.3, 36.8)
- removed the U2 at (64.8, 36.8)
- removed the U2 at (242.6, 174.0)
- removed the U2 at (135.9, 174.0)
- removed the U2 at (100.3, 174.0)
- removed the U2 at (64.8, 174.0)
- removed the U2 at (171.4, 139.7)
- removed the U3 at (211.3, 124.5)
- removed the U3 at (104.6, 124.5)
- removed the U3 at (175.8, 124.5)
- removed the U3 at (140.2, 124.5)
- removed the U3 at (69.1, 124.5)
- removed the U3 at (246.9, 90.2)
- removed the U3 at (211.3, 90.2)
- removed the U3 at (104.6, 90.2)
- removed the U3 at (175.8, 90.2)
- removed the U3 at (246.9, 158.8)
- removed the U3 at (140.2, 90.2)
- removed the U3 at (69.1, 90.2)
- removed the U3 at (246.9, 55.9)
- removed the U3 at (211.3, 55.9)
- removed the U3 at (104.6, 55.9)
- removed the U3 at (175.8, 55.9)
- removed the U3 at (140.2, 55.9)
- removed the U3 at (69.1, 55.9)
- removed the U3 at (246.9, 21.6)
- removed the U3 at (211.3, 158.8)
- removed the U3 at (211.3, 21.6)
- removed the U3 at (175.8, 21.6)
- removed the U3 at (140.2, 21.6)
- removed the U3 at (104.6, 21.6)
- removed the U3 at (69.1, 21.6)
- removed the U3 at (104.6, 158.8)
- removed the U3 at (175.8, 158.8)
- removed the U3 at (140.2, 158.8)
- removed the U3 at (69.1, 158.8)
- removed the U3 at (246.9, 124.5)
- removed the U4 at (236.2, 132.1)
- removed the U4 at (200.7, 132.1)
- removed the U4 at (129.5, 132.1)
- removed the U4 at (94.0, 132.1)
- removed the U4 at (165.1, 132.1)
- removed the U4 at (58.4, 97.8)
- removed the U4 at (236.2, 97.8)
- removed the U4 at (200.7, 97.8)
- removed the U4 at (129.5, 97.8)
- removed the U4 at (58.4, 166.4)
- removed the U4 at (94.0, 97.8)
- removed the U4 at (165.1, 97.8)
- removed the U4 at (58.4, 63.5)
- removed the U4 at (236.2, 63.5)
- removed the U4 at (200.7, 63.5)
- removed the U4 at (129.5, 63.5)
- removed the U4 at (94.0, 63.5)
- removed the U4 at (165.1, 63.5)
- removed the U4 at (236.2, 29.2)
- removed the U4 at (236.2, 166.4)
- removed the U4 at (200.7, 29.2)
- removed the U4 at (165.1, 29.2)
- removed the U4 at (129.5, 29.2)
- removed the U4 at (94.0, 29.2)
- removed the U4 at (58.4, 29.2)
- removed the U4 at (200.7, 166.4)
- removed the U4 at (129.5, 166.4)
- removed the U4 at (94.0, 166.4)
- removed the U4 at (165.1, 166.4)
- removed the U4 at (58.4, 132.1)
- removed the U5 at (200.7, 124.5)
- removed the U5 at (236.2, 124.5)
- removed the U5 at (94.0, 124.5)
- removed the U5 at (129.5, 124.5)
- removed the U5 at (165.1, 124.5)
- removed the U5 at (58.4, 90.2)
- removed the U5 at (200.7, 90.2)
- removed the U5 at (236.2, 90.2)
- removed the U5 at (94.0, 90.2)
- removed the U5 at (58.4, 158.8)
- removed the U5 at (129.5, 90.2)
- removed the U5 at (165.1, 90.2)
- removed the U5 at (58.4, 55.9)
- removed the U5 at (200.7, 55.9)
- removed the U5 at (236.2, 55.9)
- removed the U5 at (94.0, 55.9)
- removed the U5 at (129.5, 55.9)
- removed the U5 at (165.1, 55.9)
- removed the U5 at (236.2, 21.6)
- removed the U5 at (200.7, 158.8)
- removed the U5 at (200.7, 21.6)
- removed the U5 at (165.1, 21.6)
- removed the U5 at (129.5, 21.6)
- removed the U5 at (94.0, 21.6)
- removed the U5 at (58.4, 21.6)
- removed the U5 at (236.2, 158.8)
- removed the U5 at (94.0, 158.8)
- removed the U5 at (129.5, 158.8)
- removed the U5 at (165.1, 158.8)
- removed the U5 at (58.4, 124.5)
- added C1: 100N, Connector_PinHeader_2.54mm:PinHeader_1x02_P2.54mm_Vertical, B.Cu at (176.5, 176.5)
- added C1: 100N, Connector_PinHeader_2.54mm:PinHeader_1x02_P2.54mm_Vertical, B.Cu at (142.2, 142.2)
- added C1: 100N, Connector_PinHeader_2.54mm:PinHeader_1x02_P2.54mm_Vertical, B.Cu at (210.8, 142.2)
- added C1: 100N, Connector_PinHeader_2.54mm:PinHeader_1x02_P2.54mm_Vertical, B.Cu at (108.0, 142.2)
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Other:
- board text added: "by KK"

Commit message: New version of KiCAD
Other:
- net class Default removed
