File: schemat_i_inne/schemat/konwerter/konwerter/konwerter.kicad_pcb (KiCad board)
At the start: 2 copper layers, 269.2 x 182.9 mm, 455 parts, among them J1 Conn_01x06_Male, J2 Conn_01x06_Male, U1 IRF7476, U2 LM1117-1.8, U3 IRF7476, U4 IRF7476, U5 IRF7476

Commit message: Kolejna zmiana konwertera
-> poprzedni konwerter dzialal, ale nie wzialem
pod uwage droputu na MOSFETach, wiec poziomy logiczne i tak
sie nie zgadzaly

-> zmieniony konwerter z gotowa plytka, dzialajacy juz na
normalnych zasadach
Parts:
- removed the C1 at (245.1, 39.4)
- removed the C1 at (108.0, 142.2)
- removed the C1 at (73.7, 39.4)
- removed the C1 at (176.5, 108.0)
- removed the C1 at (108.0, 108.0)
- removed the C1 at (245.1, 108.0)
- removed the C1 at (142.2, 39.4)
- removed the C1 at (176.5, 39.4)
- removed the C1 at (73.7, 73.7)
- removed the C1 at (142.2, 108.0)
- removed the C1 at (245.1, 73.7)
- removed the C1 at (73.7, 176.5)
- removed the C1 at (210.8, 108.0)
- removed the C1 at (39.4, 73.7)
- removed the C1 at (73.7, 108.0)
- removed the C1 at (210.8, 142.2)
- removed the C1 at (108.0, 39.4)
- removed the C1 at (142.2, 73.7)
- removed the C1 at (73.7, 142.2)
- removed the C1 at (142.2, 142.2)
- removed the C1 at (176.5, 73.7)
- removed the C1 at (210.8, 73.7)
- removed the C1 at (39.4, 176.5)
- removed the C1 at (245.1, 142.2)
- removed the C1 at (176.5, 142.2)
- removed the C1 at (39.4, 142.2)
- removed the C1 at (39.4, 108.0)
- removed the C1 at (108.0, 73.7)
- removed the C1 at (210.8, 39.4)
- removed the C1 at (108.0, 176.5)
- removed the C1 at (210.8, 176.5)
- removed the C1 at (142.2, 176.5)
- removed the C1 at (245.1, 176.5)
- removed the C1 at (176.5, 176.5)
- removed the C1 at (39.4, 39.4)
- removed the C2 at (228.6, 39.4)
- removed the C2 at (160.0, 73.7)
- removed the C2 at (125.7, 142.2)
- removed the C2 at (57.1, 142.2)
- removed the C2 at (57.1, 108.0)
- removed the C2 at (125.7, 108.0)
- removed the C2 at (194.3, 73.7)
- removed the C2 at (160.0, 108.0)
- removed the C2 at (228.6, 108.0)
- removed the C2 at (22.9, 73.7)
- removed the C2 at (125.7, 73.7)
- removed the C2 at (22.9, 176.5)
- removed the C2 at (91.4, 142.2)
- removed the C2 at (125.7, 39.4)
- removed the C2 at (91.4, 108.0)
- removed the C2 at (57.1, 39.4)
- removed the C2 at (228.6, 142.2)
- removed the C2 at (22.9, 108.0)
- removed the C2 at (91.4, 73.7)
- removed the C2 at (228.6, 73.7)
- removed the C2 at (194.3, 39.4)
- removed the C2 at (160.0, 142.2)
- removed the C2 at (160.0, 176.5)
- removed the C2 at (160.0, 39.4)
- removed the C2 at (57.1, 73.7)
- removed the C2 at (194.3, 142.2)
- removed the C2 at (22.9, 142.2)
- removed the C2 at (194.3, 108.0)
- removed the C2 at (91.4, 39.4)
- removed the C2 at (194.3, 176.5)
- removed the C2 at (125.7, 176.5)
- removed the C2 at (91.4, 176.5)
- removed the C2 at (57.1, 176.5)
- removed the C2 at (228.6, 176.5)
- removed the C2 at (22.9, 39.4)
- removed the J1 at (222.0, 30.5)
- removed the J1 at (153.5, 30.5)
- removed the J1 at (187.8, 30.5)
- removed the J1 at (187.8, 133.3)
- removed the J1 at (153.5, 133.3)
- removed the J1 at (84.9, 64.8)
- removed the J1 at (16.3, 64.8)
- removed the J1 at (119.2, 133.3)
- removed the J1 at (50.6, 99.1)
- removed the J1 at (153.5, 99.1)
- removed the J1 at (187.8, 99.1)
- removed the J1 at (187.8, 167.6)
- removed the J1 at (16.3, 133.3)
- removed the J1 at (222.0, 64.8)
- removed the J1 at (222.0, 133.3)
- removed the J1 at (50.6, 64.8)
- removed the J1 at (84.9, 30.5)
- removed the J1 at (119.2, 64.8)
- removed the J1 at (153.5, 64.8)
- removed the J1 at (16.3, 99.1)
- removed the J1 at (187.8, 64.8)
- removed the J1 at (50.6, 133.3)
- removed the J1 at (16.3, 167.6)
- removed the J1 at (84.9, 133.3)
- removed the J1 at (84.9, 99.1)
- removed the J1 at (119.2, 30.5)
- removed the J1 at (50.6, 30.5)
- removed the J1 at (222.0, 99.1)
- removed the J1 at (119.2, 99.1)
- removed the J1 at (84.9, 167.6)
- removed the J1 at (119.2, 167.6)
- removed the J1 at (153.5, 167.6)
- removed the J1 at (50.6, 167.6)
- removed the J1 at (222.0, 167.6)
- removed the J1 at (16.3, 30.5)
- removed the J2 at (247.4, 30.5)
- removed the J2 at (41.7, 133.3)
- removed the J2 at (247.4, 64.8)
- removed the J2 at (75.9, 133.3)
- removed the J2 at (110.2, 30.5)
- removed the J2 at (178.8, 64.8)
- removed the J2 at (213.1, 133.3)
- removed the J2 at (75.9, 30.5)
- removed the J2 at (144.5, 64.8)
- removed the J2 at (110.2, 133.3)
- removed the J2 at (178.8, 30.5)
- removed the J2 at (41.7, 167.6)
- removed the J2 at (75.9, 99.1)
- removed the J2 at (213.1, 64.8)
- removed the J2 at (247.4, 133.3)
- removed the J2 at (75.9, 64.8)
- removed the J2 at (41.7, 64.8)
- removed the J2 at (110.2, 99.1)
- removed the J2 at (178.8, 99.1)
- removed the J2 at (41.7, 99.1)
- removed the J2 at (144.5, 30.5)
- removed the J2 at (213.1, 30.5)
- removed the J2 at (144.5, 167.6)
- removed the J2 at (178.8, 133.3)
- removed the J2 at (213.1, 99.1)
- removed the J2 at (110.2, 64.8)
- removed the J2 at (144.5, 99.1)
- removed the J2 at (247.4, 99.1)
- removed the J2 at (144.5, 133.3)
- removed the J2 at (213.1, 167.6)
- removed the J2 at (75.9, 167.6)
- removed the J2 at (247.4, 167.6)
- removed the J2 at (178.8, 167.6)
- removed the J2 at (110.2, 167.6)
- removed the J2 at (41.7, 30.5)
- removed the R1 at (242.6, 34.3)
- removed the R1 at (174.0, 68.6)
- removed the R1 at (139.7, 137.2)
- removed the R1 at (208.3, 102.9)
- removed the R1 at (36.8, 68.6)
- removed the R1 at (139.7, 68.6)
- removed the R1 at (105.4, 68.6)
- removed the R1 at (71.1, 34.3)
- removed the R1 at (174.0, 102.9)
- removed the R1 at (242.6, 68.6)
- removed the R1 at (105.4, 102.9)
- removed the R1 at (36.8, 171.4)
- removed the R1 at (139.7, 34.3)
- removed the R1 at (36.8, 102.9)
- removed the R1 at (36.8, 137.2)
- removed the R1 at (242.6, 102.9)
- removed the R1 at (105.4, 137.2)
- removed the R1 at (174.0, 34.3)
- removed the R1 at (71.1, 68.6)
- removed the R1 at (174.0, 137.2)
- removed the R1 at (208.3, 137.2)
- removed the R1 at (208.3, 34.3)
- removed the R1 at (208.3, 171.4)
- removed the R1 at (71.1, 102.9)
- removed the R1 at (139.7, 102.9)
- removed the R1 at (208.3, 68.6)
- removed the R1 at (242.6, 137.2)
- removed the R1 at (105.4, 34.3)
- removed the R1 at (71.1, 137.2)
- removed the R1 at (71.1, 171.4)
- removed the R1 at (105.4, 171.4)
- removed the R1 at (139.7, 171.4)
- removed the R1 at (174.0, 171.4)
- removed the R1 at (242.6, 171.4)
- removed the R1 at (36.8, 34.3)
- removed the R2 at (227.3, 16.5)
- removed the R2 at (55.9, 119.4)
- removed the R2 at (21.6, 85.1)
- removed the R2 at (158.8, 50.8)
- removed the R2 at (55.9, 85.1)
- removed the R2 at (193.0, 50.8)
- removed the R2 at (227.3, 50.8)
- removed the R2 at (21.6, 50.8)
- removed the R2 at (124.5, 119.4)
- removed the R2 at (158.8, 16.5)
- removed the R2 at (124.5, 50.8)
- removed the R2 at (21.6, 153.7)
- removed the R2 at (193.0, 16.5)
- removed the R2 at (90.2, 50.8)
- removed the R2 at (90.2, 16.5)
- removed the R2 at (227.3, 119.4)
- removed the R2 at (124.5, 85.1)
- removed the R2 at (90.2, 119.4)
- removed the R2 at (158.8, 119.4)
- removed the R2 at (90.2, 85.1)
- removed the R2 at (193.0, 119.4)
- removed the R2 at (227.3, 85.1)
- removed the R2 at (158.8, 153.7)
- removed the R2 at (55.9, 50.8)
- removed the R2 at (55.9, 16.5)
- removed the R2 at (158.8, 85.1)
- removed the R2 at (21.6, 119.4)
- removed the R2 at (193.0, 85.1)
- removed the R2 at (124.5, 16.5)
- removed the R2 at (90.2, 153.7)
- removed the R2 at (193.0, 153.7)
- removed the R2 at (227.3, 153.7)
- removed the R2 at (124.5, 153.7)
- removed the R2 at (55.9, 153.7)
- removed the R2 at (21.6, 16.5)
- removed the R3 at (240.8, 16.5)
- removed the R3 at (240.8, 85.1)
- removed the R3 at (240.8, 50.8)
- removed the R3 at (172.2, 85.1)
- removed the R3 at (137.9, 119.4)
- removed the R3 at (206.5, 85.1)
- removed the R3 at (103.6, 85.1)
- removed the R3 at (103.6, 50.8)
- removed the R3 at (35.1, 119.4)
- removed the R3 at (172.2, 16.5)
- removed the R3 at (206.5, 50.8)
- removed the R3 at (240.8, 153.7)
- removed the R3 at (69.3, 50.8)
- removed the R3 at (35.1, 50.8)
- removed the R3 at (137.9, 16.5)
- removed the R3 at (206.5, 16.5)
- removed the R3 at (69.3, 119.4)
- removed the R3 at (103.6, 16.5)
- removed the R3 at (69.3, 85.1)
- removed the R3 at (240.8, 119.4)
- removed the R3 at (69.3, 16.5)
- removed the R3 at (172.2, 119.4)
- removed the R3 at (69.3, 153.7)
- removed the R3 at (206.5, 119.4)
- removed the R3 at (137.9, 50.8)
- removed the R3 at (137.9, 85.1)
- removed the R3 at (103.6, 119.4)
- removed the R3 at (35.1, 85.1)
- removed the R3 at (172.2, 50.8)
- removed the R3 at (35.1, 153.7)
- removed the R3 at (172.2, 153.7)
- removed the R3 at (206.5, 153.7)
- removed the R3 at (103.6, 153.7)
- removed the R3 at (137.9, 153.7)
- removed the R3 at (35.1, 16.5)
- removed the R4 at (228.6, 34.3)
- removed the R4 at (57.1, 68.6)
- removed the R4 at (22.9, 102.9)
- removed the R4 at (194.3, 34.3)
- removed the R4 at (194.3, 102.9)
- removed the R4 at (125.7, 137.2)
- removed the R4 at (228.6, 68.6)
- removed the R4 at (91.4, 137.2)
- removed the R4 at (194.3, 137.2)
- removed the R4 at (228.6, 102.9)
- removed the R4 at (160.0, 34.3)
- removed the R4 at (22.9, 171.4)
- removed the R4 at (91.4, 68.6)
- removed the R4 at (57.1, 34.3)
- removed the R4 at (228.6, 137.2)
- removed the R4 at (125.7, 68.6)
- removed the R4 at (160.0, 137.2)
- removed the R4 at (91.4, 34.3)
- removed the R4 at (194.3, 68.6)
- removed the R4 at (57.1, 102.9)
- removed the R4 at (91.4, 102.9)
- removed the R4 at (125.7, 34.3)
- removed the R4 at (125.7, 171.4)
- removed the R4 at (160.0, 68.6)
- removed the R4 at (22.9, 68.6)
- removed the R4 at (160.0, 102.9)
- removed the R4 at (22.9, 137.2)
- removed the R4 at (57.1, 137.2)
- removed the R4 at (125.7, 102.9)
- removed the R4 at (194.3, 171.4)
- removed the R4 at (57.1, 171.4)
- removed the R4 at (160.0, 171.4)
- removed the R4 at (228.6, 171.4)
- removed the R4 at (91.4, 171.4)
- removed the R4 at (22.9, 34.3)
- removed the U1 at (239.3, 29.2)
- removed the U1 at (102.1, 63.5)
- removed the U1 at (33.5, 97.8)
- removed the U1 at (205.0, 132.1)
- removed the U1 at (170.7, 29.2)
- removed the U1 at (33.5, 63.5)
- removed the U1 at (136.4, 29.2)
- removed the U1 at (67.8, 132.1)
- removed the U1 at (239.3, 97.8)
- removed the U1 at (205.0, 97.8)
- removed the U1 at (239.3, 63.5)
- removed the U1 at (67.8, 166.4)
- removed the U1 at (136.4, 63.5)
- removed the U1 at (205.0, 29.2)
- removed the U1 at (136.4, 132.1)
- removed the U1 at (102.1, 132.1)
- removed the U1 at (33.5, 132.1)
- removed the U1 at (67.8, 63.5)
- removed the U1 at (205.0, 63.5)
- removed the U1 at (67.8, 29.2)
- removed the U1 at (170.7, 63.5)
- removed the U1 at (170.7, 97.8)
- removed the U1 at (33.5, 166.4)
- removed the U1 at (102.1, 97.8)
- removed the U1 at (239.3, 132.1)
- removed the U1 at (67.8, 97.8)
- removed the U1 at (102.1, 29.2)
- removed the U1 at (136.4, 97.8)
- removed the U1 at (170.7, 132.1)
- removed the U1 at (170.7, 166.4)
- removed the U1 at (205.0, 166.4)
- removed the U1 at (239.3, 166.4)
- removed the U1 at (136.4, 166.4)
- removed the U1 at (102.1, 166.4)
- removed the U1 at (33.5, 29.2)
- removed the U2 at (234.9, 36.8)
- removed the U2 at (200.7, 71.1)
- removed the U2 at (200.7, 36.8)
- removed the U2 at (63.5, 105.4)
- removed the U2 at (29.2, 139.7)
- removed the U2 at (132.1, 139.7)
- removed the U2 at (234.9, 71.1)
- removed the U2 at (63.5, 36.8)
- removed the U2 at (166.4, 36.8)
- removed the U2 at (166.4, 139.7)
- removed the U2 at (63.5, 139.7)
- removed the U2 at (29.2, 174.0)
- removed the U2 at (97.8, 36.8)
- removed the U2 at (234.9, 139.7)
- removed the U2 at (234.9, 105.4)
- removed the U2 at (29.2, 71.1)
- removed the U2 at (166.4, 71.1)
- removed the U2 at (97.8, 139.7)
- removed the U2 at (97.8, 105.4)
- removed the U2 at (29.2, 105.4)
- removed the U2 at (200.7, 139.7)
- removed the U2 at (132.1, 105.4)
- removed the U2 at (200.7, 174.0)
- removed the U2 at (200.7, 105.4)
- removed the U2 at (63.5, 71.1)
- removed the U2 at (132.1, 71.1)
- removed the U2 at (97.8, 71.1)
- removed the U2 at (132.1, 36.8)
- removed the U2 at (166.4, 105.4)
- removed the U2 at (234.9, 174.0)
- removed the U2 at (132.1, 174.0)
- removed the U2 at (63.5, 174.0)
- removed the U2 at (166.4, 174.0)
- removed the U2 at (97.8, 174.0)
- removed the U2 at (29.2, 36.8)
- removed the U3 at (239.3, 21.6)
- removed the U3 at (136.4, 21.6)
- removed the U3 at (170.7, 55.9)
- removed the U3 at (136.4, 124.5)
- removed the U3 at (67.8, 90.2)
- removed the U3 at (67.8, 21.6)
- removed the U3 at (102.1, 55.9)
- removed the U3 at (33.5, 90.2)
- removed the U3 at (239.3, 90.2)
- removed the U3 at (67.8, 124.5)
- removed the U3 at (136.4, 55.9)
- removed the U3 at (33.5, 158.8)
- removed the U3 at (136.4, 90.2)
- removed the U3 at (170.7, 124.5)
- removed the U3 at (205.0, 21.6)
- removed the U3 at (33.5, 55.9)
- removed the U3 at (102.1, 21.6)
- removed the U3 at (239.3, 55.9)
- removed the U3 at (205.0, 90.2)
- removed the U3 at (205.0, 124.5)
- removed the U3 at (170.7, 21.6)
- removed the U3 at (33.5, 124.5)
- removed the U3 at (239.3, 158.8)
- removed the U3 at (102.1, 90.2)
- removed the U3 at (170.7, 90.2)
- removed the U3 at (205.0, 55.9)
- removed the U3 at (102.1, 124.5)
- removed the U3 at (67.8, 55.9)
- removed the U3 at (239.3, 124.5)
- removed the U3 at (205.0, 158.8)
- removed the U3 at (136.4, 158.8)
- removed the U3 at (67.8, 158.8)
- removed the U3 at (170.7, 158.8)
- removed the U3 at (102.1, 158.8)
- removed the U3 at (33.5, 21.6)
- removed the U4 at (228.6, 29.2)
- removed the U4 at (91.4, 97.8)
- removed the U4 at (228.6, 63.5)
- removed the U4 at (194.3, 63.5)
- removed the U4 at (228.6, 132.1)
- removed the U4 at (22.9, 132.1)
- removed the U4 at (22.9, 97.8)
- removed the U4 at (22.9, 63.5)
- removed the U4 at (160.0, 97.8)
- removed the U4 at (125.7, 132.1)
- removed the U4 at (228.6, 97.8)
- removed the U4 at (228.6, 166.4)
- removed the U4 at (57.1, 97.8)
- removed the U4 at (125.7, 29.2)
- removed the U4 at (91.4, 29.2)
- removed the U4 at (160.0, 132.1)
- removed the U4 at (57.1, 29.2)
- removed the U4 at (194.3, 29.2)
- removed the U4 at (125.7, 97.8)
- removed the U4 at (91.4, 132.1)
- removed the U4 at (160.0, 29.2)
- removed the U4 at (91.4, 63.5)
- removed the U4 at (22.9, 166.4)
- removed the U4 at (194.3, 132.1)
- removed the U4 at (125.7, 63.5)
- removed the U4 at (57.1, 132.1)
- removed the U4 at (194.3, 97.8)
- removed the U4 at (57.1, 63.5)
- removed the U4 at (160.0, 63.5)
- removed the U4 at (194.3, 166.4)
- removed the U4 at (160.0, 166.4)
- removed the U4 at (125.7, 166.4)
- removed the U4 at (91.4, 166.4)
- removed the U4 at (57.1, 166.4)
- removed the U4 at (22.9, 29.2)
- removed the U5 at (228.6, 21.6)
- removed the U5 at (194.3, 55.9)
- removed the U5 at (194.3, 124.5)
- removed the U5 at (160.0, 21.6)
- removed the U5 at (125.7, 124.5)
- removed the U5 at (194.3, 90.2)
- removed the U5 at (228.6, 55.9)
- removed the U5 at (22.9, 55.9)
- removed the U5 at (228.6, 124.5)
- removed the U5 at (160.0, 55.9)
- removed the U5 at (57.1, 124.5)
- removed the U5 at (22.9, 158.8)
- removed the U5 at (228.6, 90.2)
- removed the U5 at (91.4, 124.5)
- removed the U5 at (57.1, 21.6)
- removed the U5 at (125.7, 90.2)
- removed the U5 at (57.1, 55.9)
- removed the U5 at (22.9, 90.2)
- removed the U5 at (91.4, 21.6)
- removed the U5 at (160.0, 124.5)
- removed the U5 at (125.7, 55.9)
- removed the U5 at (57.1, 90.2)
- removed the U5 at (194.3, 158.8)
- removed the U5 at (91.4, 90.2)
- removed the U5 at (160.0, 90.2)
- removed the U5 at (22.9, 124.5)
- removed the U5 at (194.3, 21.6)
- removed the U5 at (91.4, 55.9)
- removed the U5 at (125.7, 21.6)
- removed the U5 at (57.1, 158.8)
- removed the U5 at (125.7, 158.8)
- removed the U5 at (160.0, 158.8)
- removed the U5 at (228.6, 158.8)
- removed the U5 at (91.4, 158.8)
- removed the U5 at (22.9, 21.6)
- added C1: 100N, Connector_PinHeader_2.54mm:PinHeader_1x02_P2.54mm_Vertical, B.Cu at (146.3, 18.0)
- added C1: 100N, Connector_PinHeader_2.54mm:PinHeader_1x02_P2.54mm_Vertical, B.Cu at (31.5, 133.6)
- added C1: 100N, Connector_PinHeader_2.54mm:PinHeader_1x02_P2.54mm_Vertical, B.Cu at (87.9, 18.0)
- added C1: 100N, Connector_PinHeader_2.54mm:PinHeader_1x02_P2.54mm_Vertical, B.Cu at (202.2, 75.2)
- added C1: 100N, Connector_PinHeader_2.54mm:PinHeader_1x02_P2.54mm_Vertical, B.Cu at (87.9, 75.2)
- added C1: 100N, Connector_PinHeader_2.54mm:PinHeader_1x02_P2.54mm_Vertical, B.Cu at (174.2, 75.2)
- added C1: 100N, Connector_PinHeader_2.54mm:PinHeader_1x02_P2.54mm_Vertical, B.Cu at (260.6, 75.2)
- added C1: 100N, Connector_PinHeader_2.54mm:PinHeader_1x02_P2.54mm_Vertical, B.Cu at (232.7, 75.2)
- added C1: 100N, Connector_PinHeader_2.54mm:PinHeader_1x02_P2.54mm_Vertical, B.Cu at (232.7, 18.0)
- added C1: 100N, Connector_PinHeader_2.54mm:PinHeader_1x02_P2.54mm_Vertical, B.Cu at (174.2, 18.0)
- added C1: 100N, Connector_PinHeader_2.54mm:PinHeader_1x02_P2.54mm_Vertical, B.Cu at (31.5, 75.2)
- added C1: 100N, Connector_PinHeader_2.54mm:PinHeader_1x02_P2.54mm_Vertical, B.Cu at (174.2, 133.6)
- added C1: 100N, Connector_PinHeader_2.54mm:PinHeader_1x02_P2.54mm_Vertical, B.Cu at (59.9, 75.2)
- added C1: 100N, Connector_PinHeader_2.54mm:PinHeader_1x02_P2.54mm_Vertical, B.Cu at (146.3, 75.2)
- added C1: 100N, Connector_PinHeader_2.54mm:PinHeader_1x02_P2.54mm_Vertical, B.Cu at (260.6, 18.0)
- added C1: 100N, Connector_PinHeader_2.54mm:PinHeader_1x02_P2.54mm_Vertical, B.Cu at (202.2, 18.0)
- added C1: 100N, Connector_PinHeader_2.54mm:PinHeader_1x02_P2.54mm_Vertical, B.Cu at (87.9, 133.6)
- added C1: 100N, Connector_PinHeader_2.54mm:PinHeader_1x02_P2.54mm_Vertical, B.Cu at (146.3, 133.6)
- added C1: 100N, Connector_PinHeader_2.54mm:PinHeader_1x02_P2.54mm_Vertical, B.Cu at (115.8, 133.6)
- added C1: 100N, Connector_PinHeader_2.54mm:PinHeader_1x02_P2.54mm_Vertical, B.Cu at (59.9, 18.0)
- added C1: 100N, Connector_PinHeader_2.54mm:PinHeader_1x02_P2.54mm_Vertical, B.Cu at (202.2, 133.6)
- added C1: 100N, Connector_PinHeader_2.54mm:PinHeader_1x02_P2.54mm_Vertical, B.Cu at (31.5, 18.0)
- added C1: 100N, Connector_PinHeader_2.54mm:PinHeader_1x02_P2.54mm_Vertical, B.Cu at (59.9, 133.6)
- added C1: 100N, Connector_PinHeader_2.54mm:PinHeader_1x02_P2.54mm_Vertical, B.Cu at (260.6, 133.6)
- added C1: 100N, Connector_PinHeader_2.54mm:PinHeader_1x02_P2.54mm_Vertical, B.Cu at (232.7, 133.6)
- added C1: 100N, Connector_PinHeader_2.54mm:PinHeader_1x02_P2.54mm_Vertical, B.Cu at (115.8, 18.0)
- added C1: 100N, Connector_PinHeader_2.54mm:PinHeader_1x02_P2.54mm_Vertical, B.Cu at (115.8, 75.2)
- added C2: 2,2uF, Connector_PinHeader_2.54mm:PinHeader_1x02_P2.54mm_Vertical, B.Cu at (104.1, 133.6)
- added C2: 2,2uF, Connector_PinHeader_2.54mm:PinHeader_1x02_P2.54mm_Vertical, B.Cu at (134.6, 18.0)
- added C2: 2,2uF, Connector_PinHeader_2.54mm:PinHeader_1x02_P2.54mm_Vertical, B.Cu at (104.1, 75.2)
- added C2: 2,2uF, Connector_PinHeader_2.54mm:PinHeader_1x02_P2.54mm_Vertical, B.Cu at (134.6, 75.2)
- added C2: 2,2uF, Connector_PinHeader_2.54mm:PinHeader_1x02_P2.54mm_Vertical, B.Cu at (221.0, 75.2)
- added C2: 2,2uF, Connector_PinHeader_2.54mm:PinHeader_1x02_P2.54mm_Vertical, B.Cu at (76.2, 75.2)
- added C2: 2,2uF, Connector_PinHeader_2.54mm:PinHeader_1x02_P2.54mm_Vertical, B.Cu at (162.6, 133.6)
- added C2: 2,2uF, Connector_PinHeader_2.54mm:PinHeader_1x02_P2.54mm_Vertical, B.Cu at (19.8, 133.6)
- added C2: 2,2uF, Connector_PinHeader_2.54mm:PinHeader_1x02_P2.54mm_Vertical, B.Cu at (19.8, 18.0)
- added C2: 2,2uF, Connector_PinHeader_2.54mm:PinHeader_1x02_P2.54mm_Vertical, B.Cu at (248.9, 75.2)
- added C2: 2,2uF, Connector_PinHeader_2.54mm:PinHeader_1x02_P2.54mm_Vertical, B.Cu at (48.3, 75.2)
- added C2: 2,2uF, Connector_PinHeader_2.54mm:PinHeader_1x02_P2.54mm_Vertical, B.Cu at (221.0, 18.0)
- added C2: 2,2uF, Connector_PinHeader_2.54mm:PinHeader_1x02_P2.54mm_Vertical, B.Cu at (104.1, 18.0)
- added C2: 2,2uF, Connector_PinHeader_2.54mm:PinHeader_1x02_P2.54mm_Vertical, B.Cu at (190.5, 18.0)
- added C2: 2,2uF, Connector_PinHeader_2.54mm:PinHeader_1x02_P2.54mm_Vertical, B.Cu at (48.3, 18.0)
- added C2: 2,2uF, Connector_PinHeader_2.54mm:PinHeader_1x02_P2.54mm_Vertical, B.Cu at (48.3, 133.6)
- added C2: 2,2uF, Connector_PinHeader_2.54mm:PinHeader_1x02_P2.54mm_Vertical, B.Cu at (190.5, 133.6)
- added C2: 2,2uF, Connector_PinHeader_2.54mm:PinHeader_1x02_P2.54mm_Vertical, B.Cu at (76.2, 18.0)
- added C2: 2,2uF, Connector_PinHeader_2.54mm:PinHeader_1x02_P2.54mm_Vertical, B.Cu at (248.9, 18.0)
- added C2: 2,2uF, Connector_PinHeader_2.54mm:PinHeader_1x02_P2.54mm_Vertical, B.Cu at (76.2, 133.6)
- added C2: 2,2uF, Connector_PinHeader_2.54mm:PinHeader_1x02_P2.54mm_Vertical, B.Cu at (134.6, 133.6)
- added C2: 2,2uF, Connector_PinHeader_2.54mm:PinHeader_1x02_P2.54mm_Vertical, B.Cu at (162.6, 75.2)
- added C2: 2,2uF, Connector_PinHeader_2.54mm:PinHeader_1x02_P2.54mm_Vertical, B.Cu at (19.8, 75.2)
- added C2: 2,2uF, Connector_PinHeader_2.54mm:PinHeader_1x02_P2.54mm_Vertical, B.Cu at (221.0, 133.6)
- added C2: 2,2uF, Connector_PinHeader_2.54mm:PinHeader_1x02_P2.54mm_Vertical, B.Cu at (162.6, 18.0)
- added C2: 2,2uF, Connector_PinHeader_2.54mm:PinHeader_1x02_P2.54mm_Vertical, B.Cu at (190.5, 75.2)
- added C2: 2,2uF, Connector_PinHeader_2.54mm:PinHeader_1x02_P2.54mm_Vertical, B.Cu at (248.9, 133.6)
- added J1: Conn_01x06_Male, Connector_PinHeader_2.54mm:PinHeader_1x06_P2.54mm_Vertical, B.Cu at (132.8, 155.2)
- added J1: Conn_01x06_Male, Connector_PinHeader_2.54mm:PinHeader_1x06_P2.54mm_Vertical, B.Cu at (247.1, 39.6)
- added J1: Conn_01x06_Male, Connector_PinHeader_2.54mm:PinHeader_1x06_P2.54mm_Vertical, B.Cu at (46.5, 39.6)
- added J1: Conn_01x06_Male, Connector_PinHeader_2.54mm:PinHeader_1x06_P2.54mm_Vertical, B.Cu at (160.8, 39.6)
- added J1: Conn_01x06_Male, Connector_PinHeader_2.54mm:PinHeader_1x06_P2.54mm_Vertical, B.Cu at (46.5, 96.8)
- added J1: Conn_01x06_Male, Connector_PinHeader_2.54mm:PinHeader_1x06_P2.54mm_Vertical, B.Cu at (102.4, 39.6)
- added J1: Conn_01x06_Male, Connector_PinHeader_2.54mm:PinHeader_1x06_P2.54mm_Vertical, B.Cu at (188.7, 39.6)
- added J1: Conn_01x06_Male, Connector_PinHeader_2.54mm:PinHeader_1x06_P2.54mm_Vertical, B.Cu at (18.0, 96.8)
- added J1: Conn_01x06_Male, Connector_PinHeader_2.54mm:PinHeader_1x06_P2.54mm_Vertical, B.Cu at (102.4, 96.8)
- added J1: Conn_01x06_Male, Connector_PinHeader_2.54mm:PinHeader_1x06_P2.54mm_Vertical, B.Cu at (219.2, 96.8)
- added J1: Conn_01x06_Male, Connector_PinHeader_2.54mm:PinHeader_1x06_P2.54mm_Vertical, B.Cu at (188.7, 155.2)
- added J1: Conn_01x06_Male, Connector_PinHeader_2.54mm:PinHeader_1x06_P2.54mm_Vertical, B.Cu at (132.8, 39.6)
- added J1: Conn_01x06_Male, Connector_PinHeader_2.54mm:PinHeader_1x06_P2.54mm_Vertical, B.Cu at (74.4, 155.2)
- added J1: Conn_01x06_Male, Connector_PinHeader_2.54mm:PinHeader_1x06_P2.54mm_Vertical, B.Cu at (219.2, 39.6)
- added J1: Conn_01x06_Male, Connector_PinHeader_2.54mm:PinHeader_1x06_P2.54mm_Vertical, B.Cu at (132.8, 96.8)
- added J1: Conn_01x06_Male, Connector_PinHeader_2.54mm:PinHeader_1x06_P2.54mm_Vertical, B.Cu at (74.4, 96.8)
- added J1: Conn_01x06_Male, Connector_PinHeader_2.54mm:PinHeader_1x06_P2.54mm_Vertical, B.Cu at (160.8, 96.8)
- added J1: Conn_01x06_Male, Connector_PinHeader_2.54mm:PinHeader_1x06_P2.54mm_Vertical, B.Cu at (18.0, 39.6)
- added J1: Conn_01x06_Male, Connector_PinHeader_2.54mm:PinHeader_1x06_P2.54mm_Vertical, B.Cu at (188.7, 96.8)
- added J1: Conn_01x06_Male, Connector_PinHeader_2.54mm:PinHeader_1x06_P2.54mm_Vertical, B.Cu at (46.5, 155.2)
- added J1: Conn_01x06_Male, Connector_PinHeader_2.54mm:PinHeader_1x06_P2.54mm_Vertical, B.Cu at (160.8, 155.2)
- added J1: Conn_01x06_Male, Connector_PinHeader_2.54mm:PinHeader_1x06_P2.54mm_Vertical, B.Cu at (247.1, 155.2)
- added J1: Conn_01x06_Male, Connector_PinHeader_2.54mm:PinHeader_1x06_P2.54mm_Vertical, B.Cu at (18.0, 155.2)
- added J1: Conn_01x06_Male, Connector_PinHeader_2.54mm:PinHeader_1x06_P2.54mm_Vertical, B.Cu at (102.4, 155.2)
- added J1: Conn_01x06_Male, Connector_PinHeader_2.54mm:PinHeader_1x06_P2.54mm_Vertical, B.Cu at (247.1, 96.8)
- added J1: Conn_01x06_Male, Connector_PinHeader_2.54mm:PinHeader_1x06_P2.54mm_Vertical, B.Cu at (219.2, 155.2)
- added J1: Conn_01x06_Male, Connector_PinHeader_2.54mm:PinHeader_1x06_P2.54mm_Vertical, B.Cu at (74.4, 39.6)
- added J2: Conn_01x06_Male, Connector_PinHeader_2.54mm:PinHeader_1x06_P2.54mm_Vertical, B.Cu at (234.4, 39.6)
- added J2: Conn_01x06_Male, Connector_PinHeader_2.54mm:PinHeader_1x06_P2.54mm_Vertical, B.Cu at (61.7, 39.6)
- added J2: Conn_01x06_Male, Connector_PinHeader_2.54mm:PinHeader_1x06_P2.54mm_Vertical, B.Cu at (234.4, 96.8)
- added J2: Conn_01x06_Male, Connector_PinHeader_2.54mm:PinHeader_1x06_P2.54mm_Vertical, B.Cu at (176.0, 155.2)
- added J2: Conn_01x06_Male, Connector_PinHeader_2.54mm:PinHeader_1x06_P2.54mm_Vertical, B.Cu at (89.7, 39.6)
- added J2: Conn_01x06_Male, Connector_PinHeader_2.54mm:PinHeader_1x06_P2.54mm_Vertical, B.Cu at (117.6, 155.2)
- added J2: Conn_01x06_Male, Connector_PinHeader_2.54mm:PinHeader_1x06_P2.54mm_Vertical, B.Cu at (148.1, 155.2)
- added J2: Conn_01x06_Male, Connector_PinHeader_2.54mm:PinHeader_1x06_P2.54mm_Vertical, B.Cu at (204.0, 155.2)
- added J2: Conn_01x06_Male, Connector_PinHeader_2.54mm:PinHeader_1x06_P2.54mm_Vertical, B.Cu at (262.4, 39.6)
- added J2: Conn_01x06_Male, Connector_PinHeader_2.54mm:PinHeader_1x06_P2.54mm_Vertical, B.Cu at (262.4, 155.2)
- added J2: Conn_01x06_Male, Connector_PinHeader_2.54mm:PinHeader_1x06_P2.54mm_Vertical, B.Cu at (33.3, 155.2)
- added J2: Conn_01x06_Male, Connector_PinHeader_2.54mm:PinHeader_1x06_P2.54mm_Vertical, B.Cu at (148.1, 39.6)
- added J2: Conn_01x06_Male, Connector_PinHeader_2.54mm:PinHeader_1x06_P2.54mm_Vertical, B.Cu at (176.0, 96.8)
- added J2: Conn_01x06_Male, Connector_PinHeader_2.54mm:PinHeader_1x06_P2.54mm_Vertical, B.Cu at (262.4, 96.8)
- added J2: Conn_01x06_Male, Connector_PinHeader_2.54mm:PinHeader_1x06_P2.54mm_Vertical, B.Cu at (117.6, 96.8)
- added J2: Conn_01x06_Male, Connector_PinHeader_2.54mm:PinHeader_1x06_P2.54mm_Vertical, B.Cu at (204.0, 96.8)
- added J2: Conn_01x06_Male, Connector_PinHeader_2.54mm:PinHeader_1x06_P2.54mm_Vertical, B.Cu at (33.3, 96.8)
- added J2: Conn_01x06_Male, Connector_PinHeader_2.54mm:PinHeader_1x06_P2.54mm_Vertical, B.Cu at (117.6, 39.6)
- added J2: Conn_01x06_Male, Connector_PinHeader_2.54mm:PinHeader_1x06_P2.54mm_Vertical, B.Cu at (61.7, 155.2)
- added J2: Conn_01x06_Male, Connector_PinHeader_2.54mm:PinHeader_1x06_P2.54mm_Vertical, B.Cu at (204.0, 39.6)
- added J2: Conn_01x06_Male, Connector_PinHeader_2.54mm:PinHeader_1x06_P2.54mm_Vertical, B.Cu at (89.7, 155.2)
- added J2: Conn_01x06_Male, Connector_PinHeader_2.54mm:PinHeader_1x06_P2.54mm_Vertical, B.Cu at (33.3, 39.6)
- added J2: Conn_01x06_Male, Connector_PinHeader_2.54mm:PinHeader_1x06_P2.54mm_Vertical, B.Cu at (61.7, 96.8)
- added J2: Conn_01x06_Male, Connector_PinHeader_2.54mm:PinHeader_1x06_P2.54mm_Vertical, B.Cu at (148.1, 96.8)
- added J2: Conn_01x06_Male, Connector_PinHeader_2.54mm:PinHeader_1x06_P2.54mm_Vertical, B.Cu at (89.7, 96.8)
- added J2: Conn_01x06_Male, Connector_PinHeader_2.54mm:PinHeader_1x06_P2.54mm_Vertical, B.Cu at (234.4, 155.2)
- added J2: Conn_01x06_Male, Connector_PinHeader_2.54mm:PinHeader_1x06_P2.54mm_Vertical, B.Cu at (176.0, 39.6)
- added R1: 10K, Resistor_SMD:R_0805_2012Metric_Pad1.20x1.40mm_HandSolder, F.Cu at (224.6, 150.9)
- added R1: 10K, Resistor_SMD:R_0805_2012Metric_Pad1.20x1.40mm_HandSolder, F.Cu at (252.5, 35.3)
- added R1: 10K, Resistor_SMD:R_0805_2012Metric_Pad1.20x1.40mm_HandSolder, F.Cu at (51.8, 92.5)
- added R1: 10K, Resistor_SMD:R_0805_2012Metric_Pad1.20x1.40mm_HandSolder, F.Cu at (166.1, 150.9)
- added R1: 10K, Resistor_SMD:R_0805_2012Metric_Pad1.20x1.40mm_HandSolder, F.Cu at (23.4, 150.9)
- added R1: 10K, Resistor_SMD:R_0805_2012Metric_Pad1.20x1.40mm_HandSolder, F.Cu at (252.5, 92.5)
- added R1: 10K, Resistor_SMD:R_0805_2012Metric_Pad1.20x1.40mm_HandSolder, F.Cu at (138.2, 35.3)
- added R1: 10K, Resistor_SMD:R_0805_2012Metric_Pad1.20x1.40mm_HandSolder, F.Cu at (23.4, 92.5)
- added R1: 10K, Resistor_SMD:R_0805_2012Metric_Pad1.20x1.40mm_HandSolder, F.Cu at (107.7, 35.3)
- added R1: 10K, Resistor_SMD:R_0805_2012Metric_Pad1.20x1.40mm_HandSolder, F.Cu at (224.6, 35.3)
- added R1: 10K, Resistor_SMD:R_0805_2012Metric_Pad1.20x1.40mm_HandSolder, F.Cu at (166.1, 92.5)
- added R1: 10K, Resistor_SMD:R_0805_2012Metric_Pad1.20x1.40mm_HandSolder, F.Cu at (252.5, 150.9)
- added R1: 10K, Resistor_SMD:R_0805_2012Metric_Pad1.20x1.40mm_HandSolder, F.Cu at (224.6, 92.5)
- added R1: 10K, Resistor_SMD:R_0805_2012Metric_Pad1.20x1.40mm_HandSolder, F.Cu at (194.1, 150.9)
- added R1: 10K, Resistor_SMD:R_0805_2012Metric_Pad1.20x1.40mm_HandSolder, F.Cu at (51.8, 150.9)
- added R1: 10K, Resistor_SMD:R_0805_2012Metric_Pad1.20x1.40mm_HandSolder, F.Cu at (138.2, 150.9)
- added R1: 10K, Resistor_SMD:R_0805_2012Metric_Pad1.20x1.40mm_HandSolder, F.Cu at (194.1, 92.5)
- added R1: 10K, Resistor_SMD:R_0805_2012Metric_Pad1.20x1.40mm_HandSolder, F.Cu at (107.7, 150.9)
- added R1: 10K, Resistor_SMD:R_0805_2012Metric_Pad1.20x1.40mm_HandSolder, F.Cu at (79.8, 92.5)
- added R1: 10K, Resistor_SMD:R_0805_2012Metric_Pad1.20x1.40mm_HandSolder, F.Cu at (138.2, 92.5)
- added R1: 10K, Resistor_SMD:R_0805_2012Metric_Pad1.20x1.40mm_HandSolder, F.Cu at (79.8, 35.3)
- added R1: 10K, Resistor_SMD:R_0805_2012Metric_Pad1.20x1.40mm_HandSolder, F.Cu at (23.4, 35.3)
- added R1: 10K, Resistor_SMD:R_0805_2012Metric_Pad1.20x1.40mm_HandSolder, F.Cu at (194.1, 35.3)
- added R1: 10K, Resistor_SMD:R_0805_2012Metric_Pad1.20x1.40mm_HandSolder, F.Cu at (107.7, 92.5)
- added R1: 10K, Resistor_SMD:R_0805_2012Metric_Pad1.20x1.40mm_HandSolder, F.Cu at (79.8, 150.9)
- added R1: 10K, Resistor_SMD:R_0805_2012Metric_Pad1.20x1.40mm_HandSolder, F.Cu at (51.8, 35.3)
- added R1: 10K, Resistor_SMD:R_0805_2012Metric_Pad1.20x1.40mm_HandSolder, F.Cu at (166.1, 35.3)
- added R2: 10K, Resistor_SMD:R_0805_2012Metric_Pad1.20x1.40mm_HandSolder, F.Cu at (138.2, 101.6)
- added R2: 10K, Resistor_SMD:R_0805_2012Metric_Pad1.20x1.40mm_HandSolder, F.Cu at (252.5, 44.5)
- added R2: 10K, Resistor_SMD:R_0805_2012Metric_Pad1.20x1.40mm_HandSolder, F.Cu at (23.4, 101.6)
- added R2: 10K, Resistor_SMD:R_0805_2012Metric_Pad1.20x1.40mm_HandSolder, F.Cu at (51.8, 101.6)
- added R2: 10K, Resistor_SMD:R_0805_2012Metric_Pad1.20x1.40mm_HandSolder, F.Cu at (79.8, 160.0)
- added R2: 10K, Resistor_SMD:R_0805_2012Metric_Pad1.20x1.40mm_HandSolder, F.Cu at (51.8, 160.0)
- added R2: 10K, Resistor_SMD:R_0805_2012Metric_Pad1.20x1.40mm_HandSolder, F.Cu at (107.7, 101.6)
- added R2: 10K, Resistor_SMD:R_0805_2012Metric_Pad1.20x1.40mm_HandSolder, F.Cu at (107.7, 44.5)
- added R2: 10K, Resistor_SMD:R_0805_2012Metric_Pad1.20x1.40mm_HandSolder, F.Cu at (23.4, 160.0)
- added R2: 10K, Resistor_SMD:R_0805_2012Metric_Pad1.20x1.40mm_HandSolder, F.Cu at (79.8, 44.5)
- added R2: 10K, Resistor_SMD:R_0805_2012Metric_Pad1.20x1.40mm_HandSolder, F.Cu at (194.1, 160.0)
- added R2: 10K, Resistor_SMD:R_0805_2012Metric_Pad1.20x1.40mm_HandSolder, F.Cu at (166.1, 44.5)
- added R2: 10K, Resistor_SMD:R_0805_2012Metric_Pad1.20x1.40mm_HandSolder, F.Cu at (252.5, 101.6)
- added R2: 10K, Resistor_SMD:R_0805_2012Metric_Pad1.20x1.40mm_HandSolder, F.Cu at (224.5, 101.6)
- added R2: 10K, Resistor_SMD:R_0805_2012Metric_Pad1.20x1.40mm_HandSolder, F.Cu at (51.8, 44.5)
- added R2: 10K, Resistor_SMD:R_0805_2012Metric_Pad1.20x1.40mm_HandSolder, F.Cu at (166.1, 160.0)
- added R2: 10K, Resistor_SMD:R_0805_2012Metric_Pad1.20x1.40mm_HandSolder, F.Cu at (138.2, 160.0)
- added R2: 10K, Resistor_SMD:R_0805_2012Metric_Pad1.20x1.40mm_HandSolder, F.Cu at (166.1, 101.6)
- added R2: 10K, Resistor_SMD:R_0805_2012Metric_Pad1.20x1.40mm_HandSolder, F.Cu at (194.1, 101.6)
- added R2: 10K, Resistor_SMD:R_0805_2012Metric_Pad1.20x1.40mm_HandSolder, F.Cu at (138.2, 44.5)
- added R2: 10K, Resistor_SMD:R_0805_2012Metric_Pad1.20x1.40mm_HandSolder, F.Cu at (224.5, 160.0)
- added R2: 10K, Resistor_SMD:R_0805_2012Metric_Pad1.20x1.40mm_HandSolder, F.Cu at (23.4, 44.5)
- added R2: 10K, Resistor_SMD:R_0805_2012Metric_Pad1.20x1.40mm_HandSolder, F.Cu at (224.5, 44.5)
- added R2: 10K, Resistor_SMD:R_0805_2012Metric_Pad1.20x1.40mm_HandSolder, F.Cu at (79.8, 101.6)
- added R2: 10K, Resistor_SMD:R_0805_2012Metric_Pad1.20x1.40mm_HandSolder, F.Cu at (252.5, 160.0)
- added R2: 10K, Resistor_SMD:R_0805_2012Metric_Pad1.20x1.40mm_HandSolder, F.Cu at (194.1, 44.5)
- added R2: 10K, Resistor_SMD:R_0805_2012Metric_Pad1.20x1.40mm_HandSolder, F.Cu at (107.7, 160.0)
- added R3: 10K, Resistor_SMD:R_0805_2012Metric_Pad1.20x1.40mm_HandSolder, F.Cu at (224.5, 47.5)
- added R3: 10K, Resistor_SMD:R_0805_2012Metric_Pad1.20x1.40mm_HandSolder, F.Cu at (51.8, 163.1)
- added R3: 10K, Resistor_SMD:R_0805_2012Metric_Pad1.20x1.40mm_HandSolder, F.Cu at (252.5, 104.6)
- added R3: 10K, Resistor_SMD:R_0805_2012Metric_Pad1.20x1.40mm_HandSolder, F.Cu at (194.1, 163.1)
- added R3: 10K, Resistor_SMD:R_0805_2012Metric_Pad1.20x1.40mm_HandSolder, F.Cu at (224.5, 163.1)
- added R3: 10K, Resistor_SMD:R_0805_2012Metric_Pad1.20x1.40mm_HandSolder, F.Cu at (138.2, 47.5)
- added R3: 10K, Resistor_SMD:R_0805_2012Metric_Pad1.20x1.40mm_HandSolder, F.Cu at (51.8, 47.5)
- added R3: 10K, Resistor_SMD:R_0805_2012Metric_Pad1.20x1.40mm_HandSolder, F.Cu at (51.8, 104.6)
- added R3: 10K, Resistor_SMD:R_0805_2012Metric_Pad1.20x1.40mm_HandSolder, F.Cu at (79.8, 47.5)
- added R3: 10K, Resistor_SMD:R_0805_2012Metric_Pad1.20x1.40mm_HandSolder, F.Cu at (166.1, 163.1)
- added R3: 10K, Resistor_SMD:R_0805_2012Metric_Pad1.20x1.40mm_HandSolder, F.Cu at (23.4, 104.6)
- added R3: 10K, Resistor_SMD:R_0805_2012Metric_Pad1.20x1.40mm_HandSolder, F.Cu at (252.5, 47.5)
- added R3: 10K, Resistor_SMD:R_0805_2012Metric_Pad1.20x1.40mm_HandSolder, F.Cu at (194.1, 47.5)
- added R3: 10K, Resistor_SMD:R_0805_2012Metric_Pad1.20x1.40mm_HandSolder, F.Cu at (23.4, 163.1)
- added R3: 10K, Resistor_SMD:R_0805_2012Metric_Pad1.20x1.40mm_HandSolder, F.Cu at (107.7, 163.1)
- added R3: 10K, Resistor_SMD:R_0805_2012Metric_Pad1.20x1.40mm_HandSolder, F.Cu at (138.2, 104.6)
- added R3: 10K, Resistor_SMD:R_0805_2012Metric_Pad1.20x1.40mm_HandSolder, F.Cu at (224.5, 104.6)
- added R3: 10K, Resistor_SMD:R_0805_2012Metric_Pad1.20x1.40mm_HandSolder, F.Cu at (138.2, 163.1)
- added R3: 10K, Resistor_SMD:R_0805_2012Metric_Pad1.20x1.40mm_HandSolder, F.Cu at (79.8, 104.6)
- added R3: 10K, Resistor_SMD:R_0805_2012Metric_Pad1.20x1.40mm_HandSolder, F.Cu at (107.7, 104.6)
- added R3: 10K, Resistor_SMD:R_0805_2012Metric_Pad1.20x1.40mm_HandSolder, F.Cu at (252.5, 163.1)
- added R3: 10K, Resistor_SMD:R_0805_2012Metric_Pad1.20x1.40mm_HandSolder, F.Cu at (23.4, 47.5)
- added R3: 10K, Resistor_SMD:R_0805_2012Metric_Pad1.20x1.40mm_HandSolder, F.Cu at (194.1, 104.6)
- added R3: 10K, Resistor_SMD:R_0805_2012Metric_Pad1.20x1.40mm_HandSolder, F.Cu at (166.1, 47.5)
- added R3: 10K, Resistor_SMD:R_0805_2012Metric_Pad1.20x1.40mm_HandSolder, F.Cu at (166.1, 104.6)
- added R3: 10K, Resistor_SMD:R_0805_2012Metric_Pad1.20x1.40mm_HandSolder, F.Cu at (79.8, 163.1)
- added R3: 10K, Resistor_SMD:R_0805_2012Metric_Pad1.20x1.40mm_HandSolder, F.Cu at (107.7, 47.5)
- added R4: 10K, Resistor_SMD:R_0805_2012Metric_Pad1.20x1.40mm_HandSolder, F.Cu at (194.1, 172.2)
- added R4: 10K, Resistor_SMD:R_0805_2012Metric_Pad1.20x1.40mm_HandSolder, F.Cu at (224.5, 113.8)
- added R4: 10K, Resistor_SMD:R_0805_2012Metric_Pad1.20x1.40mm_HandSolder, F.Cu at (79.8, 172.2)
- added R4: 10K, Resistor_SMD:R_0805_2012Metric_Pad1.20x1.40mm_HandSolder, F.Cu at (79.8, 113.8)
- added R4: 10K, Resistor_SMD:R_0805_2012Metric_Pad1.20x1.40mm_HandSolder, F.Cu at (138.2, 56.6)
- added R4: 10K, Resistor_SMD:R_0805_2012Metric_Pad1.20x1.40mm_HandSolder, F.Cu at (79.8, 56.6)
- added R4: 10K, Resistor_SMD:R_0805_2012Metric_Pad1.20x1.40mm_HandSolder, F.Cu at (51.8, 113.8)
- added R4: 10K, Resistor_SMD:R_0805_2012Metric_Pad1.20x1.40mm_HandSolder, F.Cu at (107.7, 56.6)
- added R4: 10K, Resistor_SMD:R_0805_2012Metric_Pad1.20x1.40mm_HandSolder, F.Cu at (107.7, 172.2)
- added R4: 10K, Resistor_SMD:R_0805_2012Metric_Pad1.20x1.40mm_HandSolder, F.Cu at (23.4, 172.2)
- added R4: 10K, Resistor_SMD:R_0805_2012Metric_Pad1.20x1.40mm_HandSolder, F.Cu at (224.5, 172.2)
- added R4: 10K, Resistor_SMD:R_0805_2012Metric_Pad1.20x1.40mm_HandSolder, F.Cu at (51.8, 172.2)
- added R4: 10K, Resistor_SMD:R_0805_2012Metric_Pad1.20x1.40mm_HandSolder, F.Cu at (252.5, 56.6)
- added R4: 10K, Resistor_SMD:R_0805_2012Metric_Pad1.20x1.40mm_HandSolder, F.Cu at (166.1, 56.6)
- added R4: 10K, Resistor_SMD:R_0805_2012Metric_Pad1.20x1.40mm_HandSolder, F.Cu at (107.7, 113.8)
- added R4: 10K, Resistor_SMD:R_0805_2012Metric_Pad1.20x1.40mm_HandSolder, F.Cu at (224.5, 56.6)
- added R4: 10K, Resistor_SMD:R_0805_2012Metric_Pad1.20x1.40mm_HandSolder, F.Cu at (23.4, 113.8)
- added R4: 10K, Resistor_SMD:R_0805_2012Metric_Pad1.20x1.40mm_HandSolder, F.Cu at (51.8, 56.6)
- added R4: 10K, Resistor_SMD:R_0805_2012Metric_Pad1.20x1.40mm_HandSolder, F.Cu at (194.1, 113.8)
- added R4: 10K, Resistor_SMD:R_0805_2012Metric_Pad1.20x1.40mm_HandSolder, F.Cu at (166.1, 113.8)
- added R4: 10K, Resistor_SMD:R_0805_2012Metric_Pad1.20x1.40mm_HandSolder, F.Cu at (252.5, 113.8)
- added R4: 10K, Resistor_SMD:R_0805_2012Metric_Pad1.20x1.40mm_HandSolder, F.Cu at (138.2, 172.2)
- added R4: 10K, Resistor_SMD:R_0805_2012Metric_Pad1.20x1.40mm_HandSolder, F.Cu at (194.1, 56.6)
- added R4: 10K, Resistor_SMD:R_0805_2012Metric_Pad1.20x1.40mm_HandSolder, F.Cu at (138.2, 113.8)
- added R4: 10K, Resistor_SMD:R_0805_2012Metric_Pad1.20x1.40mm_HandSolder, F.Cu at (252.5, 172.2)
- added R4: 10K, Resistor_SMD:R_0805_2012Metric_Pad1.20x1.40mm_HandSolder, F.Cu at (166.1, 172.2)
- added R4: 10K, Resistor_SMD:R_0805_2012Metric_Pad1.20x1.40mm_HandSolder, F.Cu at (23.4, 56.6)
- added R5: 10K, Resistor_SMD:R_0805_2012Metric_Pad1.20x1.40mm_HandSolder, F.Cu at (198.6, 101.6)
- added R5: 10K, Resistor_SMD:R_0805_2012Metric_Pad1.20x1.40mm_HandSolder, F.Cu at (257.0, 160.0)
- added R5: 10K, Resistor_SMD:R_0805_2012Metric_Pad1.20x1.40mm_HandSolder, F.Cu at (84.3, 44.5)
- added R5: 10K, Resistor_SMD:R_0805_2012Metric_Pad1.20x1.40mm_HandSolder, F.Cu at (27.9, 101.6)
- added R5: 10K, Resistor_SMD:R_0805_2012Metric_Pad1.20x1.40mm_HandSolder, F.Cu at (257.0, 101.6)
- added R5: 10K, Resistor_SMD:R_0805_2012Metric_Pad1.20x1.40mm_HandSolder, F.Cu at (56.4, 160.0)
- added R5: 10K, Resistor_SMD:R_0805_2012Metric_Pad1.20x1.40mm_HandSolder, F.Cu at (142.7, 101.6)
- added R5: 10K, Resistor_SMD:R_0805_2012Metric_Pad1.20x1.40mm_HandSolder, F.Cu at (56.4, 44.5)
- added R5: 10K, Resistor_SMD:R_0805_2012Metric_Pad1.20x1.40mm_HandSolder, F.Cu at (198.6, 44.5)
- added R5: 10K, Resistor_SMD:R_0805_2012Metric_Pad1.20x1.40mm_HandSolder, F.Cu at (112.3, 44.5)
- added R5: 10K, Resistor_SMD:R_0805_2012Metric_Pad1.20x1.40mm_HandSolder, F.Cu at (229.1, 160.0)
- added R5: 10K, Resistor_SMD:R_0805_2012Metric_Pad1.20x1.40mm_HandSolder, F.Cu at (170.7, 160.0)
- added R5: 10K, Resistor_SMD:R_0805_2012Metric_Pad1.20x1.40mm_HandSolder, F.Cu at (142.7, 160.0)
- added R5: 10K, Resistor_SMD:R_0805_2012Metric_Pad1.20x1.40mm_HandSolder, F.Cu at (257.0, 44.5)
- added R5: 10K, Resistor_SMD:R_0805_2012Metric_Pad1.20x1.40mm_HandSolder, F.Cu at (170.7, 101.6)
- added R5: 10K, Resistor_SMD:R_0805_2012Metric_Pad1.20x1.40mm_HandSolder, F.Cu at (198.6, 160.0)
- added R5: 10K, Resistor_SMD:R_0805_2012Metric_Pad1.20x1.40mm_HandSolder, F.Cu at (142.7, 44.5)
- added R5: 10K, Resistor_SMD:R_0805_2012Metric_Pad1.20x1.40mm_HandSolder, F.Cu at (84.3, 160.0)
- added R5: 10K, Resistor_SMD:R_0805_2012Metric_Pad1.20x1.40mm_HandSolder, F.Cu at (27.9, 44.5)
- added R5: 10K, Resistor_SMD:R_0805_2012Metric_Pad1.20x1.40mm_HandSolder, F.Cu at (229.1, 44.5)
- added R5: 10K, Resistor_SMD:R_0805_2012Metric_Pad1.20x1.40mm_HandSolder, F.Cu at (112.3, 101.6)
- added R5: 10K, Resistor_SMD:R_0805_2012Metric_Pad1.20x1.40mm_HandSolder, F.Cu at (170.7, 44.5)
- added R5: 10K, Resistor_SMD:R_0805_2012Metric_Pad1.20x1.40mm_HandSolder, F.Cu at (27.9, 160.0)
- added R5: 10K, Resistor_SMD:R_0805_2012Metric_Pad1.20x1.40mm_HandSolder, F.Cu at (229.1, 101.6)
- added R5: 10K, Resistor_SMD:R_0805_2012Metric_Pad1.20x1.40mm_HandSolder, F.Cu at (56.4, 101.6)
- added R5: 10K, Resistor_SMD:R_0805_2012Metric_Pad1.20x1.40mm_HandSolder, F.Cu at (112.3, 160.0)
- added R5: 10K, Resistor_SMD:R_0805_2012Metric_Pad1.20x1.40mm_HandSolder, F.Cu at (84.3, 101.6)
- added R6: 10K, Resistor_SMD:R_0805_2012Metric_Pad1.20x1.40mm_HandSolder, F.Cu at (112.3, 47.5)
- added R6: 10K, Resistor_SMD:R_0805_2012Metric_Pad1.20x1.40mm_HandSolder, F.Cu at (257.0, 104.6)
- added R6: 10K, Resistor_SMD:R_0805_2012Metric_Pad1.20x1.40mm_HandSolder, F.Cu at (198.6, 163.1)
- added R6: 10K, Resistor_SMD:R_0805_2012Metric_Pad1.20x1.40mm_HandSolder, F.Cu at (198.6, 104.6)
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Routing:
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- removed copper zone on F.Cu, net (none)
Other:
- board size 269.2 x 182.9 mm -> 251 x 166.9 mm
- rule pad_to_mask_clearance: 0.051 -> 0
- board text removed: "Master"
- board text removed: "Slave"
