File: schemat_i_inne/schemat/RetCon.kicad_sch (KiCad schematic)
At the start: 36 parts, among them J1 Hole1, J2 Hole2, J3 Hole3, J4 Hole4, J5 programming port, J6 USB_B_Micro, SW1 SW_SPDT, SW2 Home, SW3 triggerR, SW4 Select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

Commit message: Board Completed
- sent to production
Parts:
- removed J1: Hole1, Holes:One_hole, symbol Connector:Conn_01x01_Pin
- removed J2: Hole2, Holes:One_hole, symbol Connector:Conn_01x01_Pin
- removed J3: Hole3, Holes:One_hole, symbol Connector:Conn_01x01_Pin
- removed J4: Hole4, Holes:One_hole, symbol Connector:Conn_01x01_Pin
- D1: footprint Diode_SMD:D_0603_1608Metric -> Capacitor_SMD:C_1206_3216Metric
- U2: footprint Package_TO_SOT_SMD:TO-252-2 -> Package_TO_SOT_SMD:TO-263-2
- U5: footprint (none) -> Package_SO:SO-14_3.9x8.65mm_P1.27mm
Connections:
- net at BT1.1 (+): now also SW1.1 (A); no longer SW1.3 (C)
Changed lines of the file:
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@@
+    (stroke (width 0) (type default))
+  )
+  (wire (pts (xy 33.02 182.88) (xy 33.02 185.42))
     (stroke (width 0) (type default))
   )
@@
     (stroke (width 0) (type default))
   )
-  (wire (pts (xy 30.48 180.34) (xy 33.02 180.34))
-    (stroke (width 0) (type default))
-  )
   (wire (pts (xy 120.65 81.28) (xy 125.73 81.28))
     (stroke (width 0) (type default))
@@
     (stroke (width 0) (type default))
   )
-  (wire (pts (xy 30.48 182.88) (xy 30.48 180.34))
-    (stroke (width 0) (type default))
-  )
   (wire (pts (xy 149.86 170.18) (xy 160.02 170.18))
     (stroke (width 0) (type default))
@@
   )
   (wire (pts (xy 80.01 80.01) (xy 105.41 80.01))
+    (stroke (width 0) (type default))
+  )
+  (wire (pts (xy 30.48 182.88) (xy 33.02 182.88))
     (stroke (width 0) (type default))
   )
@@
       (effects (font (size 1.27 1.27)))
     )
-    (property "Footprint" "Package_TO_SOT_SMD:TO-252-2" (at 66.675 186.69 0)
+    (property "Footprint" "Package_TO_SOT_SMD:TO-263-2" (at 66.675 186.69 0)
       (effects (font (size 1.27 1.27) italic) (justify left) hide)
     )
@@
       (effects (font (size 1.27 1.27)))
     )
-    (property "Footprint" "" (at 269.24 124.46 0)
+    (property "Footprint" "Package_SO:SO-14_3.9x8.65mm_P1.27mm" (at 269.24 124.46 0)
       (effects (font (size 1.27 1.27)) hide)
     )
@@
     )
   )
-  (symbol (lib_id "Connector:Conn_01x01_Pin") (at 252.73 48.26 0) (unit 1)
-    (in_bom yes) (on_board yes) (dnp no)
-    (property "Reference" "J3" (at 252.73 46.99 0)
-      (effects (font (size 1.27 1.27)))
-    )
-    (property "Value" "Hole3" (at 243.84 46.99 0)
-      (effects (font (size 1.27 1.27)))
-    )
-    (property "Footprint" "Holes:One_hole" (at 252.73 48.26 0)
-      (effects (font (size 1.27 1.27)) hide)
-    )
-    (property "Datasheet" "~" (at 252.73 48.26 0)
-      (effects (font (size 1.27 1.27)) hide)
-    )
-    (pin "1")
-    (instances
-      (project "schemat"
-        (path "/275aa44a-b61f-489f-9e2a-819a0fe0d1eb"
-          (reference "J3") (unit 1)
-        )
-      )
-    )
-  )
   (symbol (lib_name "GND_7") (lib_id "power:GND") (at 76.2 67.31 270) (unit 1)
     (in_bom yes) (on_board yes) (dnp no) (fields_autoplaced)
@@
       (effects (font (size 1.27 1.27)))
     )
-    (property "Footprint" "" (at 269.24 113.03 0)
+    (property "Footprint" "Package_SO:SO-14_3.9x8.65mm_P1.27mm" (at 269.24 113.03 0)
       (effects (font (size 1.27 1.27)) hide)
     )
@@
     )
   )
-  (symbol (lib_id "Connector:Conn_01x01_Pin") (at 252.73 50.8 0) (unit 1)
-    (in_bom yes) (on_board yes) (dnp no)
-    (property "Reference" "J4" (at 252.73 49.53 0)
-      (effects (font (size 1.27 1.27)))
-    )
-    (property "Value" "Hole4" (at 243.84 49.53 0)
-      (effects (font (size 1.27 1.27)))
-    )
-    (property "Footprint" "Holes:One_hole" (at 252.73 50.8 0)
-      (effects (font (size 1.27 1.27)) hide)
-    )
-    (property "Datasheet" "~" (at 252.73 50.8 0)
-      (effects (font (size 1.27 1.27)) hide)
-    )
-    (pin "1")
-    (instances
-      (project "schemat"
-        (path "/275aa44a-b61f-489f-9e2a-819a0fe0d1eb"
-          (reference "J4") (unit 1)
-        )
-      )
-    )
-  )
   (symbol (lib_id "Switch:SW_Push") (at 74.93 80.01 0) (unit 1)
     (in_bom yes) (on_board yes) (dnp no) (fields_autoplaced)
@@
       (effects (font (size 1.27 1.27)))
     )
-    (property "Footprint" "Diode_SMD:D_0603_1608Metric" (at 49.53 182.88 0)
+    (property "Footprint" "Capacitor_SMD:C_1206_3216Metric" (at 49.53 182.88 0)
       (effects (font (size 1.27 1.27)) hide)
     )
@@
     )
   )
-  (symbol (lib_id "Connector:Conn_01x01_Pin") (at 252.73 45.72 0) (unit 1)
-    (in_bom yes) (on_board yes) (dnp no)
-    (property "Reference" "J2" (at 252.73 44.45 0)
-      (effects (font (size 1.27 1.27)))
-    )
-    (property "Value" "Hole2" (at 243.84 44.45 0)
-      (effects (font (size 1.27 1.27)))
-    )
-    (property "Footprint" "Holes:One_hole" (at 252.73 45.72 0)
-      (effects (font (size 1.27 1.27)) hide)
-    )
-    (property "Datasheet" "~" (at 252.73 45.72 0)
-      (effects (font (size 1.27 1.27)) hide)
-    )
-    (pin "1")
-    (instances
-      (project "schemat"
-        (path "/275aa44a-b61f-489f-9e2a-819a0fe0d1eb"
-          (reference "J2") (unit 1)
-        )
-      )
-    )
-  )
   (symbol (lib_name "+5V_1") (lib_id "power:+5V") (at 120.65 81.28 0) (unit 1)
     (in_bom yes) (on_board yes) (dnp no) (fields_autoplaced)
@@
         )
       )
-    )
-  )
-  (symbol (lib_id "Connector:Conn_01x01_Pin") (at 252.73 43.18 0) (unit 1)
-    (in_bom yes) (on_board yes) (dnp no)
-    (property "Reference" "J1" (at 252.73 41.91 0)
-      (effects (font (size 1.27 1.27)))
-    )
-    (property "Value" "Hole1" (at 243.84 41.91 0)
-      (effects (font (size 1.27 1.27)))
-    )
-    (property "Footprint" "Holes:One_hole" (at 252.73 43.18 0)
-      (effects (font (size 1.27 1.27)) hide)
-    )
-    (property "Datasheet" "~" (at 252.73 43.18 0)
-      (effects (font (size 1.27 1.27)) hide)
-    )
-    (pin "1")
-    (instances
-      (project "schemat"
-        (path "/275aa44a-b61f-489f-9e2a-819a0fe0d1eb"
-          (reference "J1") (unit 1)
-        )
-      )
