File: schemat_i_inne/schemat/RetCon.kicad_pcb (KiCad board)
At the start: 2 copper layers, 139.5 x 70.4 mm, 36 parts, among them J1 Hole1, J2 Hole2, J3 Hole3, J4 Hole4, J5 programming port, J6 USB_B_Micro, SW1 SW_SPDT, SW2 Home, SW3 triggerR, SW4 Select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

Commit message: Board Completed
- sent to production
Parts:
- BZ1, J5, SW1: moved to B.Cu
- D1: footprint Diode_SMD:D_0603_1608Metric -> Capacitor_SMD:C_1206_3216Metric
- U2: footprint Package_TO_SOT_SMD:TO-252-2 -> Package_TO_SOT_SMD:TO-263-2
- moved D1 12.4 mm to (227.1, 106.7)
- moved L1 7.77 mm to (183.9, 61.0), turned to 0 degrees
- moved C2 7.10 mm to (204.5, 101.0)
- moved U2 4.29 mm to (211.5, 95.2)
- moved J1 1.27 mm to (207.0, 63.5)
- moved J4 1.27 mm to (120.7, 61.0)
- moved C1 1.04 mm to (219.1, 94.8)
- turned J5 to 0 degrees
- turned SW1 to 90 degrees
Connections:
- SW1 pad 1: unconnected-(SW1-A-Pad1) -> Net-(BT1-+)
- SW1 pad 3: Net-(BT1-+) -> unconnected-(SW1-C-Pad3)
Routing:
- net +5V: track 532.9 -> 561.7 mm, vias 5 -> 6
- net Net-(D1-K): track 6.15 -> 27.3 mm
- net Net-(D1-A): track 5.62 -> 18.4 mm
- net Net-(U1-AVCC): track 11.1 -> 21.3 mm
- net GND: track 186.4 -> 196.1 mm, vias 20 -> 23
- net Net-(BT1-+): track 23.4 -> 27.3 mm
- net Net-(U1-PA3): track 46.3 -> 47.0 mm
- net Net-(U1-PA1): track 107.8 -> 107.2 mm

Commit message: RetCon config file and small updates
- names of triggers and bumpers updated
- schematic, board updated
- added picture how RetCon looks in reality
Parts:
- SW3: value triggerR -> BumperR
- SW5: value triggerL -> BumperL
- SW6: value BumperL -> TriggerR
- SW7: value BumperR -> TriggerL
Changed lines of the file:
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@@
         (effects (font (size 1 1) (thickness 0.15)))
     )
-    (fp_text value "BumperL" (at 2.25 5.38988) (layer "F.Fab")
+    (fp_text value "TriggerR" (at 2.25 5.38988) (layer "F.Fab")
         (effects (font (size 1 1) (thickness 0.15)))
     )
@@
         (effects (font (size 1 1) (thickness 0.15)))
     )
-    (fp_text value "BumperR" (at 2.25 5.38988) (layer "F.Fab")
+    (fp_text value "TriggerL" (at 2.25 5.38988) (layer "F.Fab")
         (effects (font (size 1 1) (thickness 0.15)))
     )
@@
         (effects (font (size 1 1) (thickness 0.15)) (justify mirror))
     )
-    (fp_text value "triggerL" (at 2.25 -5.38988) (layer "B.Fab")
+    (fp_text value "BumperL" (at 2.25 -5.38988) (layer "B.Fab")
         (effects (font (size 1 1) (thickness 0.15)) (justify mirror))
     )
@@
         (effects (font (size 1 1) (thickness 0.15)) (justify mirror))
     )
-    (fp_text value "triggerR" (at 2.25 -5.38988) (layer "B.Fab")
+    (fp_text value "BumperR" (at 2.25 -5.38988) (layer "B.Fab")
         (effects (font (size 1 1) (thickness 0.15)) (justify mirror))
     )
@@
     (pts (xy 93.98 49.276) (xy 233.4768 49.276))
     (height -2.54)
-    (gr_text "139.4968 mm" (at 163.7284 45.586) (layer "Cmts.User")
+    (gr_text "139,4968 mm" (at 163.7284 45.586) (layer "Cmts.User")
       (effects (font (size 1 1) (thickness 0.15)))
     )
@@
     (pts (xy 233.5022 119.634) (xy 233.5022 49.276))
     (height 4.826)
-    (gr_text "70.3580 mm" (at 237.1782 84.455 90) (layer "Cmts.User")
+    (gr_text "70,3580 mm" (at 237.1782 84.455 90) (layer "Cmts.User")
       (effects (font (size 1 1) (thickness 0.15)))
     )
